File: Hardware/Motortreiber002/Stromversorgung.sch (KiCad schematic (older format))
At the start: 2 parts, among them J1 Conn_01x02

Commit message: 16 Motortreiber 1 ATXMega 128 mit USB USB Anschluss noch nicht fertig
Connections:
- net +28V: now also C1.1, J1.1 (Pin_1)
- net GND: now also C1.2, J1.2 (Pin_2)
Changed lines of the file:
@@
 $Descr A4 11693 8268
 encoding utf-8
-Sheet 2 7
+Sheet 2 19
 Title ""
 Date ""
@@
 $EndComp
 $Comp
-L power:GND #PWR0101
-U 1 1 5CAFA597
-P 1300 1450
-F 0 "#PWR0101" H 1300 1200 50  0001 C CNN
-F 1 "GND" H 1305 1277 50  0000 C CNN
-F 2 "" H 1300 1450 50  0001 C CNN
-F 3 "" H 1300 1450 50  0001 C CNN
-	1    1300 1450
-	1    0    0    -1
-$EndComp
-$Comp
-L power:GND #PWR0102
+L power:GND #PWR02
 U 1 1 5CAFA87C
 P 2150 1550
-F 0 "#PWR0102" H 2150 1300 50  0001 C CNN
+F 0 "#PWR02" H 2150 1300 50  0001 C CNN
 F 1 "GND" H 2155 1377 50  0000 C CNN
 F 2 "" H 2150 1550 50  0001 C CNN
@@
 $EndComp
 $Comp
-L power:+28V #PWR0103
+L power:+28V #PWR01
 U 1 1 5CAFAE48
 P 2150 850
-F 0 "#PWR0103" H 2150 700 50  0001 C CNN
+F 0 "#PWR01" H 2150 700 50  0001 C CNN
 F 1 "+28V" H 2165 1023 50  0000 C CNN
 F 2 "" H 2400 900 50  0001 C CNN
@@
 $EndComp
 $Comp
-L power:+5V #PWR0104
+L power:+5V #PWR03
 U 1 1 5CAFB359
 P 2900 1250
-F 0 "#PWR0104" H 2900 1100 50  0001 C CNN
+F 0 "#PWR03" H 2900 1100 50  0001 C CNN
 F 1 "+5V" H 2915 1423 50  0000 C CNN
 F 2 "" H 2900 1250 50  0001 C CNN
@@
 	1    0    0    -1
 $EndComp
+$Comp
+L power:+5VA #PWR04
+U 1 1 5CCA1750
+P 3250 1250
+F 0 "#PWR04" H 3250 1100 50  0001 C CNN
+F 1 "+5VA" H 3265 1423 50  0000 C CNN
+F 2 "" H 3250 1250 50  0001 C CNN
+F 3 "" H 3250 1250 50  0001 C CNN
+	1    3250 1250
+	1    0    0    -1
+$EndComp
+Wire Wire Line
+	2150 1550 2150 1400
+Wire Wire Line
+	2150 1050 2150 900
+Wire Wire Line
+	1300 1200 1550 1200
+Wire Wire Line
+	1550 1200 1550 900
+Wire Wire Line
+	1550 900  2150 900
+Connection ~ 2150 900
+Wire Wire Line
+	2150 900  2150 850
+Wire Wire Line
+	2150 1400 1550 1400
+Wire Wire Line
+	1550 1400 1550 1300
+Wire Wire Line
+	1550 1300 1300 1300
+Connection ~ 2150 1400
+Wire Wire Line
+	2150 1400 2150 1350
 $EndSCHEMATC

Commit message: Annotation auf Seiten bezogen
Parts:
- renumbered C1 to C201, J1 to J201
Changed lines of the file:
@@
 $EndDescr
 $Comp
-L Connector_Generic:Conn_01x02 J1
+L Connector_Generic:Conn_01x02 J201
 U 1 1 5CAF9E3E
 P 1100 1200
-F 0 "J1" H 1018 1417 50  0000 C CNN
+F 0 "J201" H 1018 1417 50  0000 C CNN
 F 1 "Conn_01x02" H 1018 1326 50  0000 C CNN
 F 2 "" H 1100 1200 50  0001 C CNN
@@
 $EndComp
 $Comp
-L Device:CP C1
+L Device:CP C201
 U 1 1 5CAFA369
 P 2150 1200
-F 0 "C1" H 2268 1246 50  0000 L CNN
+F 0 "C201" H 2268 1246 50  0000 L CNN
 F 1 "CP" H 2268 1155 50  0000 L CNN
 F 2 "" H 2188 1050 50  0001 C CNN
@@
 $EndComp
 $Comp
-L power:GND #PWR02
+L power:GND #PWR0202
 U 1 1 5CAFA87C
 P 2150 1550
-F 0 "#PWR02" H 2150 1300 50  0001 C CNN
+F 0 "#PWR0202" H 2150 1300 50  0001 C CNN
 F 1 "GND" H 2155 1377 50  0000 C CNN
 F 2 "" H 2150 1550 50  0001 C CNN
@@
 $EndComp
 $Comp
-L power:+28V #PWR01
+L power:+28V #PWR0201
 U 1 1 5CAFAE48
 P 2150 850
-F 0 "#PWR01" H 2150 700 50  0001 C CNN
+F 0 "#PWR0201" H 2150 700 50  0001 C CNN
 F 1 "+28V" H 2165 1023 50  0000 C CNN
 F 2 "" H 2400 900 50  0001 C CNN
@@
 $EndComp
 $Comp
-L power:+5V #PWR03
+L power:+5V #PWR0203
 U 1 1 5CAFB359
 P 2900 1250
-F 0 "#PWR03" H 2900 1100 50  0001 C CNN
+F 0 "#PWR0203" H 2900 1100 50  0001 C CNN
 F 1 "+5V" H 2915 1423 50  0000 C CNN
 F 2 "" H 2900 1250 50  0001 C CNN
@@
 $EndComp
 $Comp
-L power:+5VA #PWR04
+L power:+5VA #PWR0204
 U 1 1 5CCA1750
 P 3250 1250
-F 0 "#PWR04" H 3250 1100 50  0001 C CNN
+F 0 "#PWR0204" H 3250 1100 50  0001 C CNN
 F 1 "+5VA" H 3265 1423 50  0000 C CNN
 F 2 "" H 3250 1250 50  0001 C CNN
