File: Hardware/Motortreiber002/Motorteiber002.kicad_pcb (KiCad board)
At the start: 2 copper layers, 210 x 290 mm, 210 parts, among them J1001 Screw_Terminal_01x04, J1002 Screw_Terminal_01x04, J1101 Screw_Terminal_01x04, J1102 Screw_Terminal_01x04, J1201 Screw_Terminal_01x04, J1202 Screw_Terminal_01x04, J1301 Screw_Terminal_01x04, J1302 Screw_Terminal_01x04, J1401 Screw_Terminal_01x04, J1402 Screw_Terminal_01x04, J1501 Screw_Terminal_01x04, J1502 Screw_Terminal_01x04, J1601 Screw_Terminal_01x04, J1602 Screw_Terminal_01x04, J1701 Screw_Terminal_01x04, J1702 Screw_Terminal_01x04, J1801 Screw_Terminal_01x04, J1802 Screw_Terminal_01x04, J1901 Screw_Terminal_01x04, J1902 Screw_Terminal_01x04, J301 Screw_Terminal_01x04, J302 Screw_Terminal_01x04, J401 Screw_Terminal_01x04, J402 Screw_Terminal_01x04, J601 Screw_Terminal_01x04, J602 Screw_Terminal_01x04, J701 Screw_Terminal_01x04, J702 Screw_Terminal_01x04, J801 Screw_Terminal_01x04, J802 Screw_Terminal_01x04, J901 Screw_Terminal_01x04, J902 Screw_Terminal_01x04, U1001 DRV8823, U1101 DRV8823, U1201 DRV8823, U1301 DRV8823, U1401 DRV8823, U1501 DRV8823, U1601 DRV8823, U1701 DRV8823, U1801 DRV8823, U1901 DRV8823, U301 DRV8823, U401 DRV8823, U501 ADUM3160, U502 ATxmega128C3-AU, U601 DRV8823, U701 DRV8823, U801 DRV8823, U901 DRV8823

Commit message: platzierung angefangen
Parts:
- removed C1501, C1503, C301, C303, C401, C403, C601, C603, C701, C703, C801, C803, C901, C903: 100nF, Capacitor_THT:C_Disc_D8.0mm_W5.0mm_P5.00mm
- removed C1502, C302, C402, C602, C702, C802, C902: 100nF, Capacitor_SMD:C_0805_2012Metric_Pad1.15x1.40mm_HandSolder
- removed C1505, C305, C405, C605, C705, C805, C905: 100uF, Capacitor_THT:CP_Radial_D8.0mm_P3.50mm
- removed C1507, C307, C407, C607, C707, C807, C907: 10nF, Capacitor_SMD:C_0805_2012Metric
- removed C1508, C308, C408, C608, C708, C808, C908: 100nf, Capacitor_SMD:C_0805_2012Metric_Pad1.15x1.40mm_HandSolder
- removed J1501, J1502, J301, J302, J401, J402, J601, J602, J701, J702, J801, J802, J901, J902: Screw_Terminal_01x04, Connector_Phoenix_MC_HighVoltage:PhoenixContact_MCV_1,5_4-G-5.08_1x04_P5.08mm_Vertical
- removed R1501, R1502, R1503, R1504, R301, R302, R303, R304, R401, R402, R403, R404, R601, R602, R603, R604, R701, R702, R703, R704, R801, R802, R803, R804, R901, R902, R903, R904: 0R5, Resistor_THT:R_Axial_DIN0411_L9.9mm_D3.6mm_P5.08mm_Vertical
- removed U1501, U301, U401, U601, U701, U801, U901: DRV8823, Package_SO:TSSOP-48_6.1x12.5mm_P0.5mm
- added C1509: 100nF, Capacitor_THT:C_Disc_D8.0mm_W5.0mm_P5.00mm, F.Cu at (55.1, 120.4)
- added C1510: 100nF, Capacitor_SMD:C_0805_2012Metric_Pad1.15x1.40mm_HandSolder, F.Cu at (64.8, 118.6)
- added C1511: 100nF, Capacitor_THT:C_Disc_D8.0mm_W5.0mm_P5.00mm, F.Cu at (54.8, 127.0)
- added C1513: 100uF, Capacitor_THT:CP_Radial_D8.0mm_P3.50mm, F.Cu at (46.0, 125.8)
- added C1515: 10nF, Capacitor_SMD:C_0805_2012Metric, F.Cu at (64.7, 108.3)
- added C1516: 100nf, Capacitor_SMD:C_0805_2012Metric_Pad1.15x1.40mm_HandSolder, F.Cu at (64.8, 121.6)
- added C2001: 100nF, Capacitor_THT:C_Disc_D8.0mm_W5.0mm_P5.00mm, F.Cu at (173.1, 60.9)
- added C2002: 100nF, Capacitor_SMD:C_0805_2012Metric_Pad1.15x1.40mm_HandSolder, F.Cu at (183.1, 55.5)
- added C2003: 100nF, Capacitor_THT:C_Disc_D8.0mm_W5.0mm_P5.00mm, F.Cu at (173.4, 54.4)
- added C2005: 100uF, Capacitor_THT:CP_Radial_D8.0mm_P3.50mm, F.Cu at (164.3, 59.7)
- added C2007: 10nF, Capacitor_SMD:C_0805_2012Metric, F.Cu at (183.0, 42.3)
- added C2008: 100nf, Capacitor_SMD:C_0805_2012Metric_Pad1.15x1.40mm_HandSolder, F.Cu at (183.1, 52.6)
- added C2101: 100nF, Capacitor_THT:C_Disc_D8.0mm_W5.0mm_P5.00mm, F.Cu at (174.7, 90.5)
- added C2102: 100nF, Capacitor_SMD:C_0805_2012Metric_Pad1.15x1.40mm_HandSolder, F.Cu at (184.6, 85.1)
- added C2103: 100nF, Capacitor_THT:C_Disc_D8.0mm_W5.0mm_P5.00mm, F.Cu at (175.0, 83.9)
- added C2105: 100uF, Capacitor_THT:CP_Radial_D8.0mm_P3.50mm, F.Cu at (165.9, 89.3)
- added C2107: 10nF, Capacitor_SMD:C_0805_2012Metric, F.Cu at (184.6, 71.8)
- added C2108: 100nf, Capacitor_SMD:C_0805_2012Metric_Pad1.15x1.40mm_HandSolder, F.Cu at (184.6, 82.1)
- added C2201: 100nF, Capacitor_THT:C_Disc_D8.0mm_W5.0mm_P5.00mm, F.Cu at (175.7, 119.5)
- added C2202: 100nF, Capacitor_SMD:C_0805_2012Metric_Pad1.15x1.40mm_HandSolder, F.Cu at (185.6, 114.1)
- added C2203: 100nF, Capacitor_THT:C_Disc_D8.0mm_W5.0mm_P5.00mm, F.Cu at (176.0, 112.9)
- added C2205: 100uF, Capacitor_THT:CP_Radial_D8.0mm_P3.50mm, F.Cu at (166.9, 118.3)
- added C2207: 10nF, Capacitor_SMD:C_0805_2012Metric, F.Cu at (185.6, 100.8)
- added C2208: 100nf, Capacitor_SMD:C_0805_2012Metric_Pad1.15x1.40mm_HandSolder, F.Cu at (185.6, 111.1)
- added C2301: 100nF, Capacitor_THT:C_Disc_D8.0mm_W5.0mm_P5.00mm, F.Cu at (175.9, 148.6)
- added C2302: 100nF, Capacitor_SMD:C_0805_2012Metric_Pad1.15x1.40mm_HandSolder, F.Cu at (185.9, 140.2)
- added C2303: 100nF, Capacitor_THT:C_Disc_D8.0mm_W5.0mm_P5.00mm, F.Cu at (176.3, 142.0)
- added C2305: 100uF, Capacitor_THT:CP_Radial_D8.0mm_P3.50mm, F.Cu at (167.2, 147.3)
- added C2307: 10nF, Capacitor_SMD:C_0805_2012Metric, F.Cu at (185.8, 129.9)
- added C2308: 100nf, Capacitor_SMD:C_0805_2012Metric_Pad1.15x1.40mm_HandSolder, F.Cu at (185.9, 143.2)
- added C2401: 100nF, Capacitor_THT:C_Disc_D8.0mm_W5.0mm_P5.00mm, F.Cu at (176.3, 171.3)
- added C2402: 100nF, Capacitor_SMD:C_0805_2012Metric_Pad1.15x1.40mm_HandSolder, F.Cu at (185.9, 169.5)
- added C2403: 100nF, Capacitor_THT:C_Disc_D8.0mm_W5.0mm_P5.00mm, F.Cu at (175.9, 177.9)
- added C2405: 100uF, Capacitor_THT:CP_Radial_D8.0mm_P3.50mm, F.Cu at (167.2, 176.7)
- added C2407: 10nF, Capacitor_SMD:C_0805_2012Metric, F.Cu at (185.8, 159.2)
- added C2408: 100nf, Capacitor_SMD:C_0805_2012Metric_Pad1.15x1.40mm_HandSolder, F.Cu at (185.9, 172.5)
- added C2501: 100nF, Capacitor_THT:C_Disc_D8.0mm_W5.0mm_P5.00mm, F.Cu at (175.7, 203.4)
- added C2502: 100nF, Capacitor_SMD:C_0805_2012Metric_Pad1.15x1.40mm_HandSolder, F.Cu at (185.6, 195.1)
- added C2503: 100nF, Capacitor_THT:C_Disc_D8.0mm_W5.0mm_P5.00mm, F.Cu at (176.0, 196.8)
- added C2505: 100uF, Capacitor_THT:CP_Radial_D8.0mm_P3.50mm, F.Cu at (166.9, 202.2)
- added C2507: 10nF, Capacitor_SMD:C_0805_2012Metric, F.Cu at (185.6, 184.8)
- added C2508: 100nf, Capacitor_SMD:C_0805_2012Metric_Pad1.15x1.40mm_HandSolder, F.Cu at (185.6, 198.0)
- added J1503: Screw_Terminal_01x04, Connector_Phoenix_MC_HighVoltage:PhoenixContact_MCV_1,5_4-G-5.08_1x04_P5.08mm_Vertical, F.Cu at (24.0, 112.2)
- added J1504: Screw_Terminal_01x04, Connector_Phoenix_MC_HighVoltage:PhoenixContact_MCV_1,5_4-G-5.08_1x04_P5.08mm_Vertical, F.Cu at (24.0, 121.6)
- added J2001: Screw_Terminal_01x04, Connector_Phoenix_MC_HighVoltage:PhoenixContact_MCV_1,5_4-G-5.08_1x04_P5.08mm_Vertical, F.Cu at (142.3, 46.2)
- added J2002: Screw_Terminal_01x04, Connector_Phoenix_MC_HighVoltage:PhoenixContact_MCV_1,5_4-G-5.08_1x04_P5.08mm_Vertical, F.Cu at (142.3, 55.5)
- added J2101: Screw_Terminal_01x04, Connector_Phoenix_MC_HighVoltage:PhoenixContact_MCV_1,5_4-G-5.08_1x04_P5.08mm_Vertical, F.Cu at (143.9, 75.8)
- added J2102: Screw_Terminal_01x04, Connector_Phoenix_MC_HighVoltage:PhoenixContact_MCV_1,5_4-G-5.08_1x04_P5.08mm_Vertical, F.Cu at (143.9, 85.1)
- added J2201: Screw_Terminal_01x04, Connector_Phoenix_MC_HighVoltage:PhoenixContact_MCV_1,5_4-G-5.08_1x04_P5.08mm_Vertical, F.Cu at (144.9, 104.7)
- added J2202: Screw_Terminal_01x04, Connector_Phoenix_MC_HighVoltage:PhoenixContact_MCV_1,5_4-G-5.08_1x04_P5.08mm_Vertical, F.Cu at (144.9, 114.1)
- added J2301: Screw_Terminal_01x04, Connector_Phoenix_MC_HighVoltage:PhoenixContact_MCV_1,5_4-G-5.08_1x04_P5.08mm_Vertical, F.Cu at (145.1, 133.8)
- added J2302: Screw_Terminal_01x04, Connector_Phoenix_MC_HighVoltage:PhoenixContact_MCV_1,5_4-G-5.08_1x04_P5.08mm_Vertical, F.Cu at (145.1, 143.2)
- added J2401: Screw_Terminal_01x04, Connector_Phoenix_MC_HighVoltage:PhoenixContact_MCV_1,5_4-G-5.08_1x04_P5.08mm_Vertical, F.Cu at (145.1, 172.5)
- added J2402: Screw_Terminal_01x04, Connector_Phoenix_MC_HighVoltage:PhoenixContact_MCV_1,5_4-G-5.08_1x04_P5.08mm_Vertical, F.Cu at (145.1, 163.2)
- added J2501: Screw_Terminal_01x04, Connector_Phoenix_MC_HighVoltage:PhoenixContact_MCV_1,5_4-G-5.08_1x04_P5.08mm_Vertical, F.Cu at (144.9, 198.0)
- added J2502: Screw_Terminal_01x04, Connector_Phoenix_MC_HighVoltage:PhoenixContact_MCV_1,5_4-G-5.08_1x04_P5.08mm_Vertical, F.Cu at (144.9, 188.7)
- added R1505: 0R5, Resistor_THT:R_Axial_DIN0411_L9.9mm_D3.6mm_P5.08mm_Vertical, F.Cu at (32.6, 128.1)
- added R1506: 0R5, Resistor_THT:R_Axial_DIN0411_L9.9mm_D3.6mm_P5.08mm_Vertical, F.Cu at (23.0, 128.1)
- added R1507: 0R5, Resistor_THT:R_Axial_DIN0411_L9.9mm_D3.6mm_P5.08mm_Vertical, F.Cu at (55.5, 114.6)
- added R1508: 0R5, Resistor_THT:R_Axial_DIN0411_L9.9mm_D3.6mm_P5.08mm_Vertical, F.Cu at (55.5, 109.4)
- added R2001: 0R5, Resistor_THT:R_Axial_DIN0411_L9.9mm_D3.6mm_P5.08mm_Vertical, F.Cu at (141.3, 62.0)
- added R2002: 0R5, Resistor_THT:R_Axial_DIN0411_L9.9mm_D3.6mm_P5.08mm_Vertical, F.Cu at (173.8, 48.5)
- added R2003: 0R5, Resistor_THT:R_Axial_DIN0411_L9.9mm_D3.6mm_P5.08mm_Vertical, F.Cu at (173.8, 43.4)
- added R2004: 0R5, Resistor_THT:R_Axial_DIN0411_L9.9mm_D3.6mm_P5.08mm_Vertical, F.Cu at (150.9, 62.0)
- added R2101: 0R5, Resistor_THT:R_Axial_DIN0411_L9.9mm_D3.6mm_P5.08mm_Vertical, F.Cu at (152.5, 91.6)
- added R2102: 0R5, Resistor_THT:R_Axial_DIN0411_L9.9mm_D3.6mm_P5.08mm_Vertical, F.Cu at (175.3, 72.9)
- added R2103: 0R5, Resistor_THT:R_Axial_DIN0411_L9.9mm_D3.6mm_P5.08mm_Vertical, F.Cu at (175.3, 78.1)
- added R2104: 0R5, Resistor_THT:R_Axial_DIN0411_L9.9mm_D3.6mm_P5.08mm_Vertical, F.Cu at (142.8, 91.6)
- added R2201: 0R5, Resistor_THT:R_Axial_DIN0411_L9.9mm_D3.6mm_P5.08mm_Vertical, F.Cu at (143.8, 120.6)
- added R2202: 0R5, Resistor_THT:R_Axial_DIN0411_L9.9mm_D3.6mm_P5.08mm_Vertical, F.Cu at (176.3, 107.1)
- added R2203: 0R5, Resistor_THT:R_Axial_DIN0411_L9.9mm_D3.6mm_P5.08mm_Vertical, F.Cu at (176.3, 101.9)
- added R2204: 0R5, Resistor_THT:R_Axial_DIN0411_L9.9mm_D3.6mm_P5.08mm_Vertical, F.Cu at (153.5, 120.6)
- added R2301: 0R5, Resistor_THT:R_Axial_DIN0411_L9.9mm_D3.6mm_P5.08mm_Vertical, F.Cu at (176.6, 136.2)
- added R2302: 0R5, Resistor_THT:R_Axial_DIN0411_L9.9mm_D3.6mm_P5.08mm_Vertical, F.Cu at (176.6, 131.0)
- added R2303: 0R5, Resistor_THT:R_Axial_DIN0411_L9.9mm_D3.6mm_P5.08mm_Vertical, F.Cu at (153.7, 149.7)
- added R2304: 0R5, Resistor_THT:R_Axial_DIN0411_L9.9mm_D3.6mm_P5.08mm_Vertical, F.Cu at (144.1, 149.7)
- added R2401: 0R5, Resistor_THT:R_Axial_DIN0411_L9.9mm_D3.6mm_P5.08mm_Vertical, F.Cu at (176.6, 165.5)
- added R2402: 0R5, Resistor_THT:R_Axial_DIN0411_L9.9mm_D3.6mm_P5.08mm_Vertical, F.Cu at (144.1, 179.0)
- added R2403: 0R5, Resistor_THT:R_Axial_DIN0411_L9.9mm_D3.6mm_P5.08mm_Vertical, F.Cu at (176.6, 160.3)
- added R2404: 0R5, Resistor_THT:R_Axial_DIN0411_L9.9mm_D3.6mm_P5.08mm_Vertical, F.Cu at (153.7, 179.0)
- added R2501: 0R5, Resistor_THT:R_Axial_DIN0411_L9.9mm_D3.6mm_P5.08mm_Vertical, F.Cu at (176.3, 191.0)
- added R2502: 0R5, Resistor_THT:R_Axial_DIN0411_L9.9mm_D3.6mm_P5.08mm_Vertical, F.Cu at (176.3, 185.8)
- added R2503: 0R5, Resistor_THT:R_Axial_DIN0411_L9.9mm_D3.6mm_P5.08mm_Vertical, F.Cu at (143.8, 204.5)
- added R2504: 0R5, Resistor_THT:R_Axial_DIN0411_L9.9mm_D3.6mm_P5.08mm_Vertical, F.Cu at (153.5, 204.5)
- added U1502: DRV8823, Package_SO:TSSOP-48_6.1x12.5mm_P0.5mm, F.Cu at (47.9, 113.9)
- added U2001: DRV8823, Package_SO:TSSOP-48_6.1x12.5mm_P0.5mm, F.Cu at (166.2, 47.9)
- added U2101: DRV8823, Package_SO:TSSOP-48_6.1x12.5mm_P0.5mm, F.Cu at (167.7, 77.4)
- added U2201: DRV8823, Package_SO:TSSOP-48_6.1x12.5mm_P0.5mm, F.Cu at (168.7, 106.4)
- added U2301: DRV8823, Package_SO:TSSOP-48_6.1x12.5mm_P0.5mm, F.Cu at (169.0, 135.5)
- added U2401: DRV8823, Package_SO:TSSOP-48_6.1x12.5mm_P0.5mm, F.Cu at (169.0, 164.8)
- added U2501: DRV8823, Package_SO:TSSOP-48_6.1x12.5mm_P0.5mm, F.Cu at (168.7, 190.3)
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Connections:
- J1001 pad 1: /Motortreiber14/MA1 -> /Motortreiber0/MA1
- J1001 pad 2: /Motortreiber14/MA2 -> /Motortreiber0/MA2
- J1001 pad 3: /Motortreiber14/MB2 -> /Motortreiber0/MB2
- J1001 pad 4: /Motortreiber14/MB1 -> /Motortreiber0/MB1
- J1002 pad 1: /Motortreiber14/MC1 -> /Motortreiber0/MC1
- J1002 pad 2: /Motortreiber14/MC2 -> /Motortreiber0/MC2
- J1002 pad 3: /Motortreiber14/MD1 -> /Motortreiber0/MD1
- J1002 pad 4: /Motortreiber14/MD2 -> /Motortreiber0/MD2
- J1101 pad 1: /Motortreiber13/MA1 -> /Motortreiber1/MA1
- J1101 pad 2: /Motortreiber13/MA2 -> /Motortreiber1/MA2
- J1101 pad 3: /Motortreiber13/MB2 -> /Motortreiber1/MB2
- J1101 pad 4: /Motortreiber13/MB1 -> /Motortreiber1/MB1
- J1102 pad 1: /Motortreiber13/MC1 -> /Motortreiber1/MC1
- J1102 pad 2: /Motortreiber13/MC2 -> /Motortreiber1/MC2
- J1102 pad 3: /Motortreiber13/MD1 -> /Motortreiber1/MD1
- J1102 pad 4: /Motortreiber13/MD2 -> /Motortreiber1/MD2
- J1201 pad 1: /Motortreiber12/MA1 -> /Motortreiber2/MA1
- J1201 pad 2: /Motortreiber12/MA2 -> /Motortreiber2/MA2
- J1201 pad 3: /Motortreiber12/MB2 -> /Motortreiber2/MB2
- J1201 pad 4: /Motortreiber12/MB1 -> /Motortreiber2/MB1
- J1202 pad 1: /Motortreiber12/MC1 -> /Motortreiber2/MC1
- J1202 pad 2: /Motortreiber12/MC2 -> /Motortreiber2/MC2
- J1202 pad 3: /Motortreiber12/MD1 -> /Motortreiber2/MD1
- J1202 pad 4: /Motortreiber12/MD2 -> /Motortreiber2/MD2
- J1301 pad 1: /Motortreiber2/MA1 -> /Motortreiber3/MA1
- J1301 pad 2: /Motortreiber2/MA2 -> /Motortreiber3/MA2
- J1301 pad 3: /Motortreiber2/MB2 -> /Motortreiber3/MB2
- J1301 pad 4: /Motortreiber2/MB1 -> /Motortreiber3/MB1
- J1302 pad 1: /Motortreiber2/MC1 -> /Motortreiber3/MC1
- J1302 pad 2: /Motortreiber2/MC2 -> /Motortreiber3/MC2
- J1302 pad 3: /Motortreiber2/MD1 -> /Motortreiber3/MD1
- J1302 pad 4: /Motortreiber2/MD2 -> /Motortreiber3/MD2
- J1401 pad 1: /Motortreiber7/MA1 -> /Motortreiber4/MA1
- J1401 pad 2: /Motortreiber7/MA2 -> /Motortreiber4/MA2
- J1401 pad 3: /Motortreiber7/MB2 -> /Motortreiber4/MB2
- J1401 pad 4: /Motortreiber7/MB1 -> /Motortreiber4/MB1
- J1402 pad 1: /Motortreiber7/MC1 -> /Motortreiber4/MC1
- J1402 pad 2: /Motortreiber7/MC2 -> /Motortreiber4/MC2
- J1402 pad 3: /Motortreiber7/MD1 -> /Motortreiber4/MD1
- J1402 pad 4: /Motortreiber7/MD2 -> /Motortreiber4/MD2
- J1601 pad 1: /Motortreiber4/MA1 -> /Motortreiber6/MA1
- J1601 pad 2: /Motortreiber4/MA2 -> /Motortreiber6/MA2
- J1601 pad 3: /Motortreiber4/MB2 -> /Motortreiber6/MB2
- J1601 pad 4: /Motortreiber4/MB1 -> /Motortreiber6/MB1
- J1602 pad 1: /Motortreiber4/MC1 -> /Motortreiber6/MC1
- J1602 pad 2: /Motortreiber4/MC2 -> /Motortreiber6/MC2
- J1602 pad 3: /Motortreiber4/MD1 -> /Motortreiber6/MD1
- J1602 pad 4: /Motortreiber4/MD2 -> /Motortreiber6/MD2
- J1701 pad 1: /Motortreiber10/MA1 -> /Motortreiber7/MA1
- J1701 pad 2: /Motortreiber10/MA2 -> /Motortreiber7/MA2
- J1701 pad 3: /Motortreiber10/MB2 -> /Motortreiber7/MB2
- J1701 pad 4: /Motortreiber10/MB1 -> /Motortreiber7/MB1
- J1702 pad 1: /Motortreiber10/MC1 -> /Motortreiber7/MC1
- J1702 pad 2: /Motortreiber10/MC2 -> /Motortreiber7/MC2
- J1702 pad 3: /Motortreiber10/MD1 -> /Motortreiber7/MD1
- J1702 pad 4: /Motortreiber10/MD2 -> /Motortreiber7/MD2
- J1801 pad 1: /Motortreiber15/MA1 -> /Motortreiber8/MA1
- J1801 pad 2: /Motortreiber15/MA2 -> /Motortreiber8/MA2
- J1801 pad 3: /Motortreiber15/MB2 -> /Motortreiber8/MB2
- J1801 pad 4: /Motortreiber15/MB1 -> /Motortreiber8/MB1
- J1802 pad 1: /Motortreiber15/MC1 -> /Motortreiber8/MC1
- J1802 pad 2: /Motortreiber15/MC2 -> /Motortreiber8/MC2
- J1802 pad 3: /Motortreiber15/MD1 -> /Motortreiber8/MD1
- J1802 pad 4: /Motortreiber15/MD2 -> /Motortreiber8/MD2
- J1901 pad 1: /Motortreiber11/MA1 -> /Motortreiber9/MA1
- J1901 pad 2: /Motortreiber11/MA2 -> /Motortreiber9/MA2
- J1901 pad 3: /Motortreiber11/MB2 -> /Motortreiber9/MB2
- J1901 pad 4: /Motortreiber11/MB1 -> /Motortreiber9/MB1
- J1902 pad 1: /Motortreiber11/MC1 -> /Motortreiber9/MC1
- J1902 pad 2: /Motortreiber11/MC2 -> /Motortreiber9/MC2
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
Commit message: Erster Motoreiber angefangen routen
Parts:
- moved J1901 58.8 mm to (199.9, 10.0), turned to 270 degrees
- moved J2001 57.9 mm to (199.9, 40.6), turned to 270 degrees
- moved J2101 56.3 mm to (199.9, 71.0), turned to 270 degrees
- moved J2401 55.7 mm to (199.9, 162.5), turned to 270 degrees
- moved J2501 55.3 mm to (199.9, 193.0), turned to 270 degrees
- moved J2201 55.1 mm to (199.9, 101.5), turned to 270 degrees
- moved J2301 54.8 mm to (199.9, 132.0), turned to 270 degrees
- moved C1902 32.3 mm to (153.0, 10.0), turned to 90 degrees
- moved C1903 29.4 mm to (146.6, 17.7), turned to 180 degrees
- moved R1901 26.8 mm to (149.1, 7.54), turned to 180 degrees
- moved C1907 25.0 mm to (157.9, 7.80), turned to 180 degrees
- moved C1908 22.9 mm to (165.5, 11.0)
- moved C1905 22.2 mm to (179.6, 15.2), turned to 270 degrees
- moved J1801 17.8 mm to (9.42, 25.3), turned to 90 degrees
- moved J1701 17.4 mm to (9.42, 55.8), turned to 90 degrees
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Connections:
- net Net-(R1001-Pad1) renamed /Motortreiber0/MDR
- net Net-(R1002-Pad1) renamed /Motortreiber0/MAR
- net Net-(R1003-Pad2) renamed /Motortreiber0/MBR
- net Net-(R1004-Pad2) renamed /Motortreiber0/MCR
- net Net-(R1101-Pad1) renamed /Motortreiber1/MDR
- net Net-(R1102-Pad1) renamed /Motortreiber1/MAR
- net Net-(R1103-Pad2) renamed /Motortreiber1/MBR
- net Net-(R1104-Pad2) renamed /Motortreiber1/MCR
- net Net-(R1201-Pad1) renamed /Motortreiber2/MDR
- net Net-(R1202-Pad1) renamed /Motortreiber2/MAR
- net Net-(R1203-Pad2) renamed /Motortreiber2/MBR
- net Net-(R1204-Pad2) renamed /Motortreiber2/MCR
- net Net-(R1301-Pad1) renamed /Motortreiber3/MDR
- net Net-(R1302-Pad1) renamed /Motortreiber3/MAR
- net Net-(R1303-Pad2) renamed /Motortreiber3/MBR
- net Net-(R1304-Pad2) renamed /Motortreiber3/MCR
- net Net-(R1401-Pad1) renamed /Motortreiber4/MDR
- net Net-(R1402-Pad1) renamed /Motortreiber4/MAR
- net Net-(R1403-Pad2) renamed /Motortreiber4/MBR
- net Net-(R1404-Pad2) renamed /Motortreiber4/MCR
- net Net-(R1505-Pad1) renamed /Motortreiber5/MDR
- net Net-(R1506-Pad1) renamed /Motortreiber5/MAR
- net Net-(R1507-Pad2) renamed /Motortreiber5/MBR
- net Net-(R1508-Pad2) renamed /Motortreiber5/MCR
- net Net-(R1601-Pad1) renamed /Motortreiber6/MDR
- net Net-(R1602-Pad1) renamed /Motortreiber6/MAR
- net Net-(R1603-Pad2) renamed /Motortreiber6/MBR
- net Net-(R1604-Pad2) renamed /Motortreiber6/MCR
- net Net-(R1701-Pad1) renamed /Motortreiber7/MDR
- net Net-(R1702-Pad1) renamed /Motortreiber7/MAR
- net Net-(R1703-Pad2) renamed /Motortreiber7/MBR
- net Net-(R1704-Pad2) renamed /Motortreiber7/MCR
- net Net-(R1801-Pad1) renamed /Motortreiber8/MDR
- net Net-(R1802-Pad1) renamed /Motortreiber8/MAR
- net Net-(R1803-Pad2) renamed /Motortreiber8/MBR
- net Net-(R1804-Pad2) renamed /Motortreiber8/MCR
- net Net-(R1901-Pad1) renamed /Motortreiber9/MDR
- net Net-(R1902-Pad1) renamed /Motortreiber9/MAR
- net Net-(R1903-Pad2) renamed /Motortreiber9/MBR
- net Net-(R1904-Pad2) renamed /Motortreiber9/MCR
- net Net-(R2001-Pad1) renamed /Motortreiber10/MDR
- net Net-(R2002-Pad1) renamed /Motortreiber10/MAR
- net Net-(R2003-Pad2) renamed /Motortreiber10/MBR
- net Net-(R2004-Pad2) renamed /Motortreiber10/MCR
- net Net-(R2101-Pad1) renamed /Motortreiber11/MDR
- net Net-(R2102-Pad1) renamed /Motortreiber11/MAR
- net Net-(R2103-Pad2) renamed /Motortreiber11/MBR
- net Net-(R2104-Pad2) renamed /Motortreiber11/MCR
- net Net-(R2201-Pad1) renamed /Motortreiber12/MDR
- net Net-(R2202-Pad1) renamed /Motortreiber12/MAR
- net Net-(R2203-Pad2) renamed /Motortreiber12/MBR
- net Net-(R2204-Pad2) renamed /Motortreiber12/MCR
- net Net-(R2301-Pad1) renamed /Motortreiber13/MDR
- net Net-(R2302-Pad1) renamed /Motortreiber13/MAR
- net Net-(R2303-Pad2) renamed /Motortreiber13/MBR
- net Net-(R2304-Pad2) renamed /Motortreiber13/MCR
- net Net-(R2401-Pad1) renamed /Motortreiber14/MDR
- net Net-(R2402-Pad1) renamed /Motortreiber14/MAR
- net Net-(R2403-Pad2) renamed /Motortreiber14/MBR
- net Net-(R2404-Pad2) renamed /Motortreiber14/MCR
- net Net-(R2501-Pad1) renamed /Motortreiber15/MDR
- net Net-(R2502-Pad1) renamed /Motortreiber15/MAR
- net Net-(R2503-Pad2) renamed /Motortreiber15/MBR
- net Net-(R2504-Pad2) renamed /Motortreiber15/MCR
Routing:
- net +28V: track 0.00 -> 71.6 mm
- net /Motortreiber9/MA1: track 0.00 -> 44.9 mm, vias 0 -> 1
- net /Motortreiber9/MA2: track 0.00 -> 41.7 mm, vias 0 -> 1
- net /Motortreiber9/MB2: track 0.00 -> 25.7 mm
- net /Motortreiber9/MB1: track 0.00 -> 24.0 mm
- net Net-(C1908-Pad1): track 0.00 -> 18.0 mm
- net /Motortreiber9/MAR: track 0.00 -> 13.7 mm, vias 0 -> 1
- net Net-(C1907-Pad2): track 0.00 -> 6.99 mm
- net Net-(C1907-Pad1): track 0.00 -> 6.88 mm
- net Net-(C1902-Pad1): track 0.00 -> 4.47 mm
Other:
- net class Motor added: clearance 0.2, trace_width 1, via_dia 1.5, via_drill 0.8

Commit message: Kondensatoren auf SMD geaendert
Parts:
- added C1004: 1nF 25V, Capacitor_SMD:C_0201_0603Metric, F.Cu at (-10.9, 264.1)
- added C1006: 1nF 25V, Capacitor_SMD:C_0201_0603Metric, F.Cu at (-17.4, 264.1)
- added C1104: 1nF 25V, Capacitor_SMD:C_0201_0603Metric, F.Cu at (254.9, 38.9)
- added C1106: 1nF 25V, Capacitor_SMD:C_0201_0603Metric, F.Cu at (261.4, 38.9)
- added C1204: 1nF 25V, Capacitor_SMD:C_0201_0603Metric, F.Cu at (237.6, 27.9)
- added C1206: 1nF 25V, Capacitor_SMD:C_0201_0603Metric, F.Cu at (244.2, 27.9)
- added C1304: 1nF 25V, Capacitor_SMD:C_0201_0603Metric, F.Cu at (237.6, 38.9)
- added C1306: 1nF 25V, Capacitor_SMD:C_0201_0603Metric, F.Cu at (244.2, 38.9)
- added C1404: 1nF 25V, Capacitor_SMD:C_0201_0603Metric, F.Cu at (254.9, 27.9)
- added C1406: 1nF 25V, Capacitor_SMD:C_0201_0603Metric, F.Cu at (261.4, 27.9)
- added C1512: 1nF 25V, Capacitor_SMD:C_0201_0603Metric, F.Cu at (237.6, 49.9)
- added C1514: 1nF 25V, Capacitor_SMD:C_0201_0603Metric, F.Cu at (244.2, 49.9)
- added C1604: 1nF 25V, Capacitor_SMD:C_0201_0603Metric, F.Cu at (278.7, 49.9)
- added C1606: 1nF 25V, Capacitor_SMD:C_0201_0603Metric, F.Cu at (272.1, 49.9)
- added C1704: 1nF 25V, Capacitor_SMD:C_0201_0603Metric, F.Cu at (261.4, 60.9)
- added C1706: 1nF 25V, Capacitor_SMD:C_0201_0603Metric, F.Cu at (254.9, 60.9)
- added C1804: 1nF 25V, Capacitor_SMD:C_0201_0603Metric, F.Cu at (289.4, 27.9)
- added C1806: 1nF 25V, Capacitor_SMD:C_0201_0603Metric, F.Cu at (295.9, 27.9)
- added C1904: 1nF 25V, Capacitor_SMD:C_0201_0603Metric, F.Cu at (155.5, -8.11)
- added C1906: 1nF 25V, Capacitor_SMD:C_0201_0603Metric, F.Cu at (148.9, -8.11)
- added C2004: 1nF 25V, Capacitor_SMD:C_0201_0603Metric, F.Cu at (261.4, 49.9)
- added C2006: 1nF 25V, Capacitor_SMD:C_0201_0603Metric, F.Cu at (254.9, 49.9)
- added C2104: 1nF 25V, Capacitor_SMD:C_0201_0603Metric, F.Cu at (244.2, 60.9)
- added C2106: 1nF 25V, Capacitor_SMD:C_0201_0603Metric, F.Cu at (237.6, 60.9)
- added C2204: 1nF 25V, Capacitor_SMD:C_0201_0603Metric, F.Cu at (289.4, 60.9)
- added C2206: 1nF 25V, Capacitor_SMD:C_0201_0603Metric, F.Cu at (295.9, 60.9)
- added C2304: 1nF 25V, Capacitor_SMD:C_0201_0603Metric, F.Cu at (289.4, 49.9)
- added C2306: 1nF 25V, Capacitor_SMD:C_0201_0603Metric, F.Cu at (295.9, 49.9)
- added C2404: 1nF 25V, Capacitor_SMD:C_0201_0603Metric, F.Cu at (289.4, 38.9)
- added C2406: 1nF 25V, Capacitor_SMD:C_0201_0603Metric, F.Cu at (295.9, 38.9)
- added C2504: 1nF 25V, Capacitor_SMD:C_0201_0603Metric, F.Cu at (272.1, 60.9)
- added C2506: 1nF 25V, Capacitor_SMD:C_0201_0603Metric, F.Cu at (278.7, 60.9)
- C1002, C1102, C1202, C1302, C1402, C1510, C1602, C1702, C1802, C1902, C2002, C2102, C2202, C2302, C2402, C2502: value 100nF -> 100nF 6,3V; footprint Capacitor_SMD:C_0805_2012Metric_Pad1.15x1.40mm_HandSolder -> Capacitor_SMD:C_0201_0603Metric
- C1005, C1105, C1205, C1305, C1405, C1513, C1605, C1705, C1805, C1905, C2005, C2105, C2205, C2305, C2405, C2505: value 100uF -> 33uF 35V; footprint Capacitor_THT:CP_Radial_D8.0mm_P3.50mm -> Capacitor_THT:CP_Radial_D5.0mm_P2.00mm
- C1007, C1107, C1207, C1307, C1407, C1515, C1607, C1707, C1807, C1907, C2007, C2107, C2207, C2307, C2407, C2507: value 10nF -> 10nF 50V; footprint Capacitor_SMD:C_0805_2012Metric -> Capacitor_SMD:C_0402_1005Metric
- C1008, C1108, C1208, C1308, C1408, C1516, C1608, C1708, C1808, C1908, C2008, C2108, C2208, C2308, C2408, C2508: value 100nf -> 100nF 16V; footprint Capacitor_SMD:C_0805_2012Metric_Pad1.15x1.40mm_HandSolder -> Capacitor_SMD:C_0402_1005Metric
- moved C1908 11.7 mm to (161.8, -0.08)
- moved C1905 7.41 mm to (185.9, 11.3)
- moved C1903 4.02 mm to (145.3, 13.9)
- moved R1903 2.54 mm to (169.4, 27.9)
- turned C1901 to 0 degrees
Routing:
- net +28V: track 71.6 -> 274.7 mm
- net /Motortreiber9/MC1: track 0.00 -> 33.5 mm, vias 0 -> 1
- net /Motortreiber9/MC2: track 0.00 -> 27.6 mm, vias 0 -> 1
- net /Motortreiber9/MD1: track 0.00 -> 21.9 mm
- net /Motortreiber9/MD2: track 0.00 -> 20.3 mm
- net /Motortreiber9/MCR: track 0.00 -> 9.75 mm
- net Net-(C1908-Pad1): track 18.0 -> 12.0 mm
- net /Motortreiber9/MA2: track 41.7 -> 43.8 mm
- net /Motortreiber9/MA1: track 44.9 -> 46.9 mm

Commit message: weiteres routing
Parts:
- moved C1906 16.7 mm to (152.4, 8.27), turned to 90 degrees
- moved C1904 16.6 mm to (153.2, 8.30), turned to 90 degrees
- moved C1908 11.2 mm to (159.0, 10.8)
- moved C1907 4.34 mm to (159.0, 12.0)
- moved C1902 2.04 mm to (154.2, 8.32)
Connections:
- C1004 pad 2: Net-(C1004-Pad2) -> GND
- C1104 pad 2: Net-(C1104-Pad2) -> GND
- C1204 pad 2: Net-(C1204-Pad2) -> GND
- C1304 pad 2: Net-(C1304-Pad2) -> GND
- C1404 pad 2: Net-(C1404-Pad2) -> GND
- C1512 pad 2: Net-(C1512-Pad2) -> GND
- C1604 pad 2: Net-(C1604-Pad2) -> GND
- C1704 pad 2: Net-(C1704-Pad2) -> GND
- C1804 pad 2: Net-(C1804-Pad2) -> GND
- C1904 pad 2: Net-(C1904-Pad2) -> GND
- C2004 pad 2: Net-(C2004-Pad2) -> GND
- C2104 pad 2: Net-(C2104-Pad2) -> GND
- C2204 pad 2: Net-(C2204-Pad2) -> GND
- C2304 pad 2: Net-(C2304-Pad2) -> GND
- C2404 pad 2: Net-(C2404-Pad2) -> GND
- C2504 pad 2: Net-(C2504-Pad2) -> GND
Routing:
- net +28V: track 274.7 -> 295.3 mm
- net /Motortreiber9/MB1: track 24.0 -> 40.8 mm, vias 0 -> 1
- net /Motortreiber9/MB2: track 25.7 -> 40.7 mm, vias 0 -> 1
- net /Motortreiber9/MDR: track 0.00 -> 13.0 mm
- net /Motortreiber9/MD2: track 20.3 -> 32.1 mm, vias 0 -> 1
- net Net-(C1908-Pad1): track 12.0 -> 3.65 mm
- net /Motortreiber9/Steuer6: track 0.00 -> 7.71 mm
- net /Motortreiber9/MD1: track 21.9 -> 29.5 mm, vias 0 -> 1
- net /Motortreiber9/Steuer5: track 0.00 -> 7.22 mm
- net /Motortreiber9/MBR: track 0.00 -> 4.99 mm
- net Net-(C1907-Pad1): track 6.88 -> 1.96 mm
- net Net-(C1907-Pad2): track 6.99 -> 2.26 mm
- net /Motortreiber9/MAR: track 13.7 -> 10.4 mm, vias 1 -> 0
- net Net-(C1902-Pad1): track 4.47 -> 6.63 mm
- net /Motortreiber9/MC2: track 27.6 -> 26.2 mm

Commit message: 16 Motortreiber
Parts:
- removed C1101, C1103, C1201, C1203, C1301, C1303, C1401, C1403, C1509, C1511, C1601, C1603, C1701, C1703, C1801, C1803, C2001, C2003, C2101, C2103, C2201, C2203, C2301, C2303, C2401, C2403, C2501, C2503: 100nF, Capacitor_THT:C_Disc_D8.0mm_W5.0mm_P5.00mm
- removed C1102, C1202, C1302, C1402, C1510, C1602, C1702, C1802, C2002, C2102, C2202, C2302, C2402, C2502: 100nF 6,3V, Capacitor_SMD:C_0201_0603Metric
- removed C1104, C1106, C1204, C1206, C1304, C1306, C1404, C1406, C1512, C1514, C1604, C1606, C1704, C1706, C1804, C1806, C2004, C2006, C2104, C2106, C2204, C2206, C2304, C2306, C2404, C2406, C2504, C2506: 1nF 25V, Capacitor_SMD:C_0201_0603Metric
- removed C1105, C1205, C1305, C1405, C1513, C1605, C1705, C1805, C2005, C2105, C2205, C2305, C2405, C2505: 33uF 35V, Capacitor_THT:CP_Radial_D5.0mm_P2.00mm
- removed C1107, C1207, C1307, C1407, C1515, C1607, C1707, C1807, C2007, C2107, C2207, C2307, C2407, C2507: 10nF 50V, Capacitor_SMD:C_0402_1005Metric
- removed C1108, C1208, C1308, C1408, C1516, C1608, C1708, C1808, C2008, C2108, C2208, C2308, C2408, C2508: 100nF 16V, Capacitor_SMD:C_0402_1005Metric
- removed the C1902 at (154.2, 8.32)
- removed the C1904 at (153.2, 8.30)
- removed the C1906 at (152.4, 8.27)
- removed J1101, J1102, J1201, J1202, J1301, J1302, J1401, J1402, J1503, J1504, J1601, J1602, J1701, J1702, J1801, J1802, J2001, J2002, J2101, J2102, J2201, J2202, J2301, J2302, J2401, J2402, J2501, J2502: Screw_Terminal_01x04, Connector_Phoenix_MC_HighVoltage:PhoenixContact_MCV_1,5_4-G-5.08_1x04_P5.08mm_Vertical
- removed R1001, R1101, R1102, R1103, R1104, R1201, R1202, R1203, R1204, R1301, R1302, R1303, R1304, R1401, R1402, R1403, R1404, R1505, R1506, R1507, R1508, R1601, R1602, R1603, R1604, R1701, R1702, R1703, R1704, R1801, R1802, R1803, R1804, R2001, R2002, R2003, R2004, R2101, R2102, R2103, R2104, R2201, R2202, R2203, R2204, R2301, R2302, R2303, R2304, R2401, R2402, R2403, R2404, R2501, R2502, R2503, R2504: 0R5, Resistor_THT:R_Axial_DIN0411_L9.9mm_D3.6mm_P5.08mm_Vertical
- removed U1101, U1201, U1301, U1401, U1502, U1601, U1701, U1801, U2001, U2101, U2201, U2301, U2401, U2501: DRV8823, Package_SO:TSSOP-48_6.1x12.5mm_P0.5mm
- removed U501: ADUM3160, Package_SO:SOIC-16W_7.5x10.3mm_P1.27mm
- removed U502: ATxmega128C3-AU, Package_QFP:TQFP-64_14x14mm_P0.8mm
- added C1901: 100nF, Capacitor_THT:C_Disc_D8.0mm_W5.0mm_P5.00mm, F.Cu at (42.1, 26.2)
- added C1901: 100nF, Capacitor_THT:C_Disc_D8.0mm_W5.0mm_P5.00mm, F.Cu at (167.8, 163.8)
- added C1901: 100nF, Capacitor_THT:C_Disc_D8.0mm_W5.0mm_P5.00mm, F.Cu at (167.8, 133.8)
- added C1901: 100nF, Capacitor_THT:C_Disc_D8.0mm_W5.0mm_P5.00mm, F.Cu at (167.8, 103.8)
- added C1901: 100nF, Capacitor_THT:C_Disc_D8.0mm_W5.0mm_P5.00mm, F.Cu at (167.8, 73.8)
- added C1901: 100nF, Capacitor_THT:C_Disc_D8.0mm_W5.0mm_P5.00mm, F.Cu at (167.8, 43.8)
- added C1901: 100nF, Capacitor_THT:C_Disc_D8.0mm_W5.0mm_P5.00mm, F.Cu at (42.1, 56.2)
- added C1901: 100nF, Capacitor_THT:C_Disc_D8.0mm_W5.0mm_P5.00mm, F.Cu at (42.1, 86.2)
- added C1901: 100nF, Capacitor_THT:C_Disc_D8.0mm_W5.0mm_P5.00mm, F.Cu at (42.1, 116.2)
- added C1901: 100nF, Capacitor_THT:C_Disc_D8.0mm_W5.0mm_P5.00mm, F.Cu at (42.1, 146.2)
- added C1901: 100nF, Capacitor_THT:C_Disc_D8.0mm_W5.0mm_P5.00mm, F.Cu at (42.1, 176.2)
- added C1901: 100nF, Capacitor_THT:C_Disc_D8.0mm_W5.0mm_P5.00mm, F.Cu at (42.1, 206.2)
- added C1901: 100nF, Capacitor_THT:C_Disc_D8.0mm_W5.0mm_P5.00mm, F.Cu at (167.8, 223.8)
- added C1901: 100nF, Capacitor_THT:C_Disc_D8.0mm_W5.0mm_P5.00mm, F.Cu at (167.8, 193.8)
- added C1902: 100nF 6,3V, Capacitor_SMD:C_0201_0603Metric, F.Cu at (57.5, 32.5)
- added C1902: 100nF 6,3V, Capacitor_SMD:C_0201_0603Metric, F.Cu at (152.5, 157.5)
- added C1902: 100nF 6,3V, Capacitor_SMD:C_0201_0603Metric, F.Cu at (152.5, 127.5)
- added C1902: 100nF 6,3V, Capacitor_SMD:C_0201_0603Metric, F.Cu at (152.5, 97.5)
- added C1902: 100nF 6,3V, Capacitor_SMD:C_0201_0603Metric, F.Cu at (152.5, 67.5)
- added C1902: 100nF 6,3V, Capacitor_SMD:C_0201_0603Metric, F.Cu at (152.5, 37.5)
- added C1902: 100nF 6,3V, Capacitor_SMD:C_0201_0603Metric, F.Cu at (152.5, 7.50)
- added C1902: 100nF 6,3V, Capacitor_SMD:C_0201_0603Metric, F.Cu at (57.5, 62.5)
- added C1902: 100nF 6,3V, Capacitor_SMD:C_0201_0603Metric, F.Cu at (57.5, 92.5)
- added C1902: 100nF 6,3V, Capacitor_SMD:C_0201_0603Metric, F.Cu at (57.5, 122.5)
- added C1902: 100nF 6,3V, Capacitor_SMD:C_0201_0603Metric, F.Cu at (57.5, 152.5)
- added C1902: 100nF 6,3V, Capacitor_SMD:C_0201_0603Metric, F.Cu at (57.5, 182.5)
- added C1902: 100nF 6,3V, Capacitor_SMD:C_0201_0603Metric, F.Cu at (57.5, 212.5)
- added C1902: 100nF 6,3V, Capacitor_SMD:C_0201_0603Metric, F.Cu at (152.5, 217.5)
- added C1902: 100nF 6,3V, Capacitor_SMD:C_0201_0603Metric, F.Cu at (152.5, 187.5)
- added C1903: 100nF, Capacitor_THT:C_Disc_D8.0mm_W5.0mm_P5.00mm, F.Cu at (64.7, 26.1)
- added C1903: 100nF, Capacitor_THT:C_Disc_D8.0mm_W5.0mm_P5.00mm, F.Cu at (145.3, 163.9)
- added C1903: 100nF, Capacitor_THT:C_Disc_D8.0mm_W5.0mm_P5.00mm, F.Cu at (145.3, 133.9)
- added C1903: 100nF, Capacitor_THT:C_Disc_D8.0mm_W5.0mm_P5.00mm, F.Cu at (145.3, 103.9)
- added C1903: 100nF, Capacitor_THT:C_Disc_D8.0mm_W5.0mm_P5.00mm, F.Cu at (145.3, 73.9)
- added C1903: 100nF, Capacitor_THT:C_Disc_D8.0mm_W5.0mm_P5.00mm, F.Cu at (145.3, 43.9)
- added C1903: 100nF, Capacitor_THT:C_Disc_D8.0mm_W5.0mm_P5.00mm, F.Cu at (64.7, 56.1)
- added C1903: 100nF, Capacitor_THT:C_Disc_D8.0mm_W5.0mm_P5.00mm, F.Cu at (64.7, 86.1)
- added C1903: 100nF, Capacitor_THT:C_Disc_D8.0mm_W5.0mm_P5.00mm, F.Cu at (64.7, 116.1)
- added C1903: 100nF, Capacitor_THT:C_Disc_D8.0mm_W5.0mm_P5.00mm, F.Cu at (64.7, 146.1)
- added C1903: 100nF, Capacitor_THT:C_Disc_D8.0mm_W5.0mm_P5.00mm, F.Cu at (64.7, 176.1)
- added C1903: 100nF, Capacitor_THT:C_Disc_D8.0mm_W5.0mm_P5.00mm, F.Cu at (64.7, 206.1)
- added C1903: 100nF, Capacitor_THT:C_Disc_D8.0mm_W5.0mm_P5.00mm, F.Cu at (145.3, 223.9)
- added C1903: 100nF, Capacitor_THT:C_Disc_D8.0mm_W5.0mm_P5.00mm, F.Cu at (145.3, 193.9)
- added C1904: 1nF 25V, Capacitor_SMD:C_0201_0603Metric, B.Cu at (57.0, 32.8)
- added C1904: 1nF 25V, Capacitor_SMD:C_0201_0603Metric, B.Cu at (153.0, 157.2)
- added C1904: 1nF 25V, Capacitor_SMD:C_0201_0603Metric, B.Cu at (153.0, 127.2)
- added C1904: 1nF 25V, Capacitor_SMD:C_0201_0603Metric, B.Cu at (153.0, 97.2)
- added C1904: 1nF 25V, Capacitor_SMD:C_0201_0603Metric, B.Cu at (153.0, 67.2)
- added C1904: 1nF 25V, Capacitor_SMD:C_0201_0603Metric, B.Cu at (153.0, 37.2)
- added C1904: 1nF 25V, Capacitor_SMD:C_0201_0603Metric, B.Cu at (153.0, 7.20)
- added C1904: 1nF 25V, Capacitor_SMD:C_0201_0603Metric, B.Cu at (57.0, 62.8)
- added C1904: 1nF 25V, Capacitor_SMD:C_0201_0603Metric, B.Cu at (57.0, 92.8)
- added C1904: 1nF 25V, Capacitor_SMD:C_0201_0603Metric, B.Cu at (57.0, 122.8)
- added C1904: 1nF 25V, Capacitor_SMD:C_0201_0603Metric, B.Cu at (57.0, 152.8)
- added C1904: 1nF 25V, Capacitor_SMD:C_0201_0603Metric, B.Cu at (57.0, 182.8)
- added C1904: 1nF 25V, Capacitor_SMD:C_0201_0603Metric, B.Cu at (57.0, 212.8)
- added C1904: 1nF 25V, Capacitor_SMD:C_0201_0603Metric, B.Cu at (153.0, 217.2)
- added C1904: 1nF 25V, Capacitor_SMD:C_0201_0603Metric, B.Cu at (153.0, 187.2)
- added C1905: 33uF 35V, Capacitor_THT:CP_Radial_D5.0mm_P2.00mm, F.Cu at (24.1, 28.6)
- added C1905: 33uF 35V, Capacitor_THT:CP_Radial_D5.0mm_P2.00mm, F.Cu at (185.9, 161.3)
- added C1905: 33uF 35V, Capacitor_THT:CP_Radial_D5.0mm_P2.00mm, F.Cu at (185.9, 131.3)
- added C1905: 33uF 35V, Capacitor_THT:CP_Radial_D5.0mm_P2.00mm, F.Cu at (185.9, 101.3)
- added C1905: 33uF 35V, Capacitor_THT:CP_Radial_D5.0mm_P2.00mm, F.Cu at (185.9, 71.3)
- added C1905: 33uF 35V, Capacitor_THT:CP_Radial_D5.0mm_P2.00mm, F.Cu at (185.9, 41.4)
- added C1905: 33uF 35V, Capacitor_THT:CP_Radial_D5.0mm_P2.00mm, F.Cu at (24.1, 58.6)
- added C1905: 33uF 35V, Capacitor_THT:CP_Radial_D5.0mm_P2.00mm, F.Cu at (24.1, 88.7)
- added C1905: 33uF 35V, Capacitor_THT:CP_Radial_D5.0mm_P2.00mm, F.Cu at (24.1, 118.7)
- added C1905: 33uF 35V, Capacitor_THT:CP_Radial_D5.0mm_P2.00mm, F.Cu at (24.1, 148.7)
- added C1905: 33uF 35V, Capacitor_THT:CP_Radial_D5.0mm_P2.00mm, F.Cu at (24.1, 178.7)
- added C1905: 33uF 35V, Capacitor_THT:CP_Radial_D5.0mm_P2.00mm, F.Cu at (24.1, 208.7)
- added C1905: 33uF 35V, Capacitor_THT:CP_Radial_D5.0mm_P2.00mm, F.Cu at (185.9, 221.3)
- added C1905: 33uF 35V, Capacitor_THT:CP_Radial_D5.0mm_P2.00mm, F.Cu at (185.9, 191.3)
- added C1906: 1nF 25V, Capacitor_SMD:C_0201_0603Metric, B.Cu at (58.0, 32.8)
- added C1906: 1nF 25V, Capacitor_SMD:C_0201_0603Metric, B.Cu at (152.0, 157.2)
- added C1906: 1nF 25V, Capacitor_SMD:C_0201_0603Metric, B.Cu at (152.0, 127.2)
- added C1906: 1nF 25V, Capacitor_SMD:C_0201_0603Metric, B.Cu at (152.0, 97.2)
- added C1906: 1nF 25V, Capacitor_SMD:C_0201_0603Metric, B.Cu at (152.0, 67.2)
- added C1906: 1nF 25V, Capacitor_SMD:C_0201_0603Metric, B.Cu at (152.0, 37.2)
- added C1906: 1nF 25V, Capacitor_SMD:C_0201_0603Metric, B.Cu at (152.0, 7.18)
- added C1906: 1nF 25V, Capacitor_SMD:C_0201_0603Metric, B.Cu at (58.0, 62.8)
- added C1906: 1nF 25V, Capacitor_SMD:C_0201_0603Metric, B.Cu at (58.0, 92.8)
- added C1906: 1nF 25V, Capacitor_SMD:C_0201_0603Metric, B.Cu at (58.0, 122.8)
- added C1906: 1nF 25V, Capacitor_SMD:C_0201_0603Metric, B.Cu at (58.0, 152.8)
- added C1906: 1nF 25V, Capacitor_SMD:C_0201_0603Metric, B.Cu at (58.0, 182.8)
- added C1906: 1nF 25V, Capacitor_SMD:C_0201_0603Metric, B.Cu at (58.0, 212.8)
- added C1906: 1nF 25V, Capacitor_SMD:C_0201_0603Metric, B.Cu at (152.0, 217.2)
- added C1906: 1nF 25V, Capacitor_SMD:C_0201_0603Metric, B.Cu at (152.0, 187.2)
- added C1907: 10nF 50V, Capacitor_SMD:C_0402_1005Metric, F.Cu at (47.0, 32.0)
- added C1907: 10nF 50V, Capacitor_SMD:C_0402_1005Metric, F.Cu at (163.0, 158.0)
- added C1907: 10nF 50V, Capacitor_SMD:C_0402_1005Metric, F.Cu at (163.0, 128.0)
- added C1907: 10nF 50V, Capacitor_SMD:C_0402_1005Metric, F.Cu at (163.0, 98.0)
- added C1907: 10nF 50V, Capacitor_SMD:C_0402_1005Metric, F.Cu at (163.0, 68.0)
- added C1907: 10nF 50V, Capacitor_SMD:C_0402_1005Metric, F.Cu at (163.0, 38.0)
- added C1907: 10nF 50V, Capacitor_SMD:C_0402_1005Metric, F.Cu at (47.0, 62.0)
- added C1907: 10nF 50V, Capacitor_SMD:C_0402_1005Metric, F.Cu at (47.0, 92.0)
- added C1907: 10nF 50V, Capacitor_SMD:C_0402_1005Metric, F.Cu at (47.0, 122.0)
- added C1907: 10nF 50V, Capacitor_SMD:C_0402_1005Metric, F.Cu at (47.0, 152.0)
- added C1907: 10nF 50V, Capacitor_SMD:C_0402_1005Metric, F.Cu at (47.0, 182.0)
- added C1907: 10nF 50V, Capacitor_SMD:C_0402_1005Metric, F.Cu at (47.0, 212.0)
- added C1907: 10nF 50V, Capacitor_SMD:C_0402_1005Metric, F.Cu at (163.0, 218.0)
- added C1907: 10nF 50V, Capacitor_SMD:C_0402_1005Metric, F.Cu at (163.0, 188.0)
- added C1908: 100nF 16V, Capacitor_SMD:C_0402_1005Metric, F.Cu at (46.0, 34.0)
- added C1908: 100nF 16V, Capacitor_SMD:C_0402_1005Metric, F.Cu at (164.0, 156.0)
- added C1908: 100nF 16V, Capacitor_SMD:C_0402_1005Metric, F.Cu at (164.0, 126.0)
- added C1908: 100nF 16V, Capacitor_SMD:C_0402_1005Metric, F.Cu at (164.0, 96.0)
- added C1908: 100nF 16V, Capacitor_SMD:C_0402_1005Metric, F.Cu at (164.0, 66.0)
- added C1908: 100nF 16V, Capacitor_SMD:C_0402_1005Metric, F.Cu at (164.0, 36.0)
- added C1908: 100nF 16V, Capacitor_SMD:C_0402_1005Metric, F.Cu at (46.0, 64.0)
- added C1908: 100nF 16V, Capacitor_SMD:C_0402_1005Metric, F.Cu at (46.0, 94.0)
- added C1908: 100nF 16V, Capacitor_SMD:C_0402_1005Metric, F.Cu at (46.0, 124.0)
- added C1908: 100nF 16V, Capacitor_SMD:C_0402_1005Metric, F.Cu at (46.0, 154.0)
- added C1908: 100nF 16V, Capacitor_SMD:C_0402_1005Metric, F.Cu at (46.0, 184.0)
- added C1908: 100nF 16V, Capacitor_SMD:C_0402_1005Metric, F.Cu at (46.0, 214.0)
- added C1908: 100nF 16V, Capacitor_SMD:C_0402_1005Metric, F.Cu at (164.0, 216.0)
- added C1908: 100nF 16V, Capacitor_SMD:C_0402_1005Metric, F.Cu at (164.0, 186.0)
- added J1901: Screw_Terminal_01x04, Connector_Phoenix_MC_HighVoltage:PhoenixContact_MCV_1,5_4-G-5.08_1x04_P5.08mm_Vertical, F.Cu at (10.1, 30.0)
- added J1901: Screw_Terminal_01x04, Connector_Phoenix_MC_HighVoltage:PhoenixContact_MCV_1,5_4-G-5.08_1x04_P5.08mm_Vertical, F.Cu at (199.9, 160.0)
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Connections:
- C1002 pad 1: Net-(C1002-Pad1) -> Net-(C1902-Pad1)
- C1004 pad 1: /Motortreiber0/Steuer5 -> /Steuer5
- C1006 pad 1: /Motortreiber0/Steuer6 -> /Steuer6
- C1007 pad 1: Net-(C1007-Pad1) -> Net-(C1907-Pad1)
- C1007 pad 2: Net-(C1007-Pad2) -> Net-(C1907-Pad2)
- C1008 pad 1: Net-(C1008-Pad1) -> Net-(C1908-Pad1)
- J1002 pad 1: /Motortreiber0/MC1 -> /Motortreiber9/MC1
- J1002 pad 2: /Motortreiber0/MC2 -> /Motortreiber9/MC2
- J1002 pad 3: /Motortreiber0/MD1 -> /Motortreiber9/MD1
- J1002 pad 4: /Motortreiber0/MD2 -> /Motortreiber9/MD2
- R1004 pad 2: /Motortreiber0/MCR -> /Motortreiber9/MCR
- U1001 pad 16: Net-(C1002-Pad1) -> Net-(C1902-Pad1)
- U1001 pad 17: /Motortreiber0/Steuer5 -> /Steuer5
- U1001 pad 18: /Motortreiber0/Steuer6 -> /Steuer6
- U1001 pad 19: Net-(U1001-Pad19) -> Net-(U1901-Pad19)
- U1001 pad 20: /Motortreiber0/MD2 -> /Motortreiber9/MD2
- U1001 pad 21: /Motortreiber0/MDR -> /Motortreiber9/MDR
- U1001 pad 22: /Motortreiber0/MD1 -> /Motortreiber9/MD1
- U1001 pad 25: /Motortreiber0/MC2 -> /Motortreiber9/MC2
- U1001 pad 26: /Motortreiber0/MCR -> /Motortreiber9/MCR
- U1001 pad 27: /Motortreiber0/MC1 -> /Motortreiber9/MC1
- U1001 pad 28: Net-(U1001-Pad28) -> Net-(U1901-Pad28)
- U1001 pad 29: Net-(U1001-Pad29) -> Net-(U1901-Pad29)
- U1001 pad 31: /Motortreiber0/Steuer2 -> /Steuer2
- U1001 pad 32: Net-(U1001-Pad32) -> Net-(U1901-Pad32)
- U1001 pad 33: /Motortreiber0/Steuer3 -> /Steuer3
- U1001 pad 40: Net-(U1001-Pad40) -> Net-(U1901-Pad40)
- U1001 pad 41: Net-(U1001-Pad41) -> Net-(U1901-Pad41)
- U1001 pad 42: /Motortreiber0/Steuer1 -> /Steuer1
- U1001 pad 43: /Motortreiber0/Steuer0 -> /Steuer0
- U1001 pad 44: Net-(U1001-Pad44) -> Net-(U1901-Pad44)
- U1001 pad 45: /Motortreiber0/Steuer4 -> /Steuer4
- U1001 pad 6: Net-(U1001-Pad6) -> Net-(U1901-Pad6)
- U1001 pad 7: Net-(C1007-Pad1) -> Net-(C1907-Pad1)
- U1001 pad 8: Net-(C1007-Pad2) -> Net-(C1907-Pad2)
- U1001 pad 9: Net-(C1008-Pad1) -> Net-(C1908-Pad1)
- U1901 pad 17: /Motortreiber9/Steuer5 -> /Steuer5
- U1901 pad 18: /Motortreiber9/Steuer6 -> /Steuer6
- U1901 pad 31: /Motortreiber9/Steuer2 -> /Steuer2
- U1901 pad 33: /Motortreiber9/Steuer3 -> /Steuer3
- U1901 pad 42: /Motortreiber9/Steuer1 -> /Steuer1
- U1901 pad 43: /Motortreiber9/Steuer0 -> /Steuer0
- U1901 pad 45: /Motortreiber9/Steuer4 -> /Steuer4
Routing:
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