File: Hardware/Motortreiber002/Motorteiber002.kicad_pcb (KiCad board)
At the start: 2 copper layers, 210 x 290 mm, 240 parts, among them J1001 Screw_Terminal_01x04, J1002 Screw_Terminal_01x04, J1901 Screw_Terminal_01x04, J1902 Screw_Terminal_01x04, U1001 DRV8823, U1901 DRV8823

Commit message: Layout 16 Motortreiber grob fertig
Parts:
- removed the C1901 at (42.1, 26.2)
- removed the C1901 at (167.8, 163.8)
- removed the C1901 at (167.8, 133.8)
- removed the C1901 at (167.8, 103.8)
- removed the C1901 at (167.8, 73.8)
- removed the C1901 at (167.8, 43.8)
- removed the C1901 at (42.1, 56.2)
- removed the C1901 at (42.1, 86.2)
- removed the C1901 at (42.1, 116.2)
- removed the C1901 at (42.1, 146.2)
- removed the C1901 at (42.1, 176.2)
- removed the C1901 at (42.1, 206.2)
- removed the C1901 at (167.8, 223.8)
- removed the C1901 at (167.8, 193.8)
- removed the C1902 at (57.5, 32.5)
- removed the C1902 at (152.5, 157.5)
- removed the C1902 at (152.5, 127.5)
- removed the C1902 at (152.5, 97.5)
- removed the C1902 at (152.5, 67.5)
- removed the C1902 at (152.5, 37.5)
- removed the C1902 at (57.5, 62.5)
- removed the C1902 at (57.5, 92.5)
- removed the C1902 at (57.5, 122.5)
- removed the C1902 at (57.5, 152.5)
- removed the C1902 at (57.5, 182.5)
- removed the C1902 at (57.5, 212.5)
- removed the C1902 at (152.5, 217.5)
- removed the C1902 at (152.5, 187.5)
- removed the C1903 at (64.7, 26.1)
- removed the C1903 at (145.3, 163.9)
- removed the C1903 at (145.3, 133.9)
- removed the C1903 at (145.3, 103.9)
- removed the C1903 at (145.3, 73.9)
- removed the C1903 at (145.3, 43.9)
- removed the C1903 at (64.7, 56.1)
- removed the C1903 at (64.7, 86.1)
- removed the C1903 at (64.7, 116.1)
- removed the C1903 at (64.7, 146.1)
- removed the C1903 at (64.7, 176.1)
- removed the C1903 at (64.7, 206.1)
- removed the C1903 at (145.3, 223.9)
- removed the C1903 at (145.3, 193.9)
- removed the C1904 at (57.0, 32.8)
- removed the C1904 at (153.0, 157.2)
- removed the C1904 at (153.0, 127.2)
- removed the C1904 at (153.0, 97.2)
- removed the C1904 at (153.0, 67.2)
- removed the C1904 at (153.0, 37.2)
- removed the C1904 at (57.0, 62.8)
- removed the C1904 at (57.0, 92.8)
- removed the C1904 at (57.0, 122.8)
- removed the C1904 at (57.0, 152.8)
- removed the C1904 at (57.0, 182.8)
- removed the C1904 at (57.0, 212.8)
- removed the C1904 at (153.0, 217.2)
- removed the C1904 at (153.0, 187.2)
- removed the C1905 at (24.1, 28.6)
- removed the C1905 at (185.9, 161.3)
- removed the C1905 at (185.9, 131.3)
- removed the C1905 at (185.9, 101.3)
- removed the C1905 at (185.9, 71.3)
- removed the C1905 at (185.9, 41.4)
- removed the C1905 at (24.1, 58.6)
- removed the C1905 at (24.1, 88.7)
- removed the C1905 at (24.1, 118.7)
- removed the C1905 at (24.1, 148.7)
- removed the C1905 at (24.1, 178.7)
- removed the C1905 at (24.1, 208.7)
- removed the C1905 at (185.9, 221.3)
- removed the C1905 at (185.9, 191.3)
- removed the C1906 at (58.0, 32.8)
- removed the C1906 at (152.0, 157.2)
- removed the C1906 at (152.0, 127.2)
- removed the C1906 at (152.0, 97.2)
- removed the C1906 at (152.0, 67.2)
- removed the C1906 at (152.0, 37.2)
- removed the C1906 at (58.0, 62.8)
- removed the C1906 at (58.0, 92.8)
- removed the C1906 at (58.0, 122.8)
- removed the C1906 at (58.0, 152.8)
- removed the C1906 at (58.0, 182.8)
- removed the C1906 at (58.0, 212.8)
- removed the C1906 at (152.0, 217.2)
- removed the C1906 at (152.0, 187.2)
- removed the C1907 at (47.0, 32.0)
- removed the C1907 at (163.0, 158.0)
- removed the C1907 at (163.0, 128.0)
- removed the C1907 at (163.0, 98.0)
- removed the C1907 at (163.0, 68.0)
- removed the C1907 at (163.0, 38.0)
- removed the C1907 at (47.0, 62.0)
- removed the C1907 at (47.0, 92.0)
- removed the C1907 at (47.0, 122.0)
- removed the C1907 at (47.0, 152.0)
- removed the C1907 at (47.0, 182.0)
- removed the C1907 at (47.0, 212.0)
- removed the C1907 at (163.0, 218.0)
- removed the C1907 at (163.0, 188.0)
- removed the C1908 at (46.0, 34.0)
- removed the C1908 at (164.0, 156.0)
- removed the C1908 at (164.0, 126.0)
- removed the C1908 at (164.0, 96.0)
- removed the C1908 at (164.0, 66.0)
- removed the C1908 at (164.0, 36.0)
- removed the C1908 at (46.0, 64.0)
- removed the C1908 at (46.0, 94.0)
- removed the C1908 at (46.0, 124.0)
- removed the C1908 at (46.0, 154.0)
- removed the C1908 at (46.0, 184.0)
- removed the C1908 at (46.0, 214.0)
- removed the C1908 at (164.0, 216.0)
- removed the C1908 at (164.0, 186.0)
- removed the J1901 at (10.1, 30.0)
- removed the J1901 at (199.9, 160.0)
- removed the J1901 at (199.9, 130.0)
- removed the J1901 at (199.9, 100.0)
- removed the J1901 at (199.9, 70.0)
- removed the J1901 at (199.9, 40.0)
- removed the J1901 at (10.1, 60.0)
- removed the J1901 at (10.1, 90.0)
- removed the J1901 at (10.1, 120.0)
- removed the J1901 at (10.1, 150.0)
- removed the J1901 at (10.1, 180.0)
- removed the J1901 at (10.1, 210.0)
- removed the J1901 at (199.9, 220.0)
- removed the J1901 at (199.9, 190.0)
- removed the J1902 at (83.7, 14.7)
- removed the J1902 at (126.3, 175.3)
- removed the J1902 at (126.3, 145.3)
- removed the J1902 at (126.3, 115.3)
- removed the J1902 at (126.3, 85.3)
- removed the J1902 at (126.3, 55.3)
- removed the J1902 at (83.7, 44.7)
- removed the J1902 at (83.7, 74.7)
- removed the J1902 at (83.7, 104.7)
- removed the J1902 at (83.7, 134.7)
- removed the J1902 at (83.7, 164.7)
- removed the J1902 at (83.7, 194.7)
- removed the J1902 at (126.3, 235.3)
- removed the J1902 at (126.3, 205.3)
- removed the R1901 at (60.9, 32.5)
- removed the R1901 at (149.1, 187.5)
- removed the R1901 at (149.1, 157.5)
- removed the R1901 at (149.1, 127.5)
- removed the R1901 at (149.1, 97.5)
- removed the R1901 at (149.1, 67.5)
- removed the R1901 at (149.1, 37.5)
- removed the R1901 at (60.9, 62.5)
- removed the R1901 at (60.9, 92.5)
- removed the R1901 at (60.9, 122.5)
- removed the R1901 at (60.9, 152.5)
- removed the R1901 at (60.9, 182.5)
- removed the R1901 at (60.9, 212.5)
- removed the R1901 at (60.9, 242.5)
- removed the R1901 at (149.1, 217.5)
- removed the R1902 at (43.1, 32.5)
- removed the R1902 at (166.9, 157.5)
- removed the R1902 at (166.9, 127.5)
- removed the R1902 at (166.9, 97.5)
- removed the R1902 at (166.9, 67.5)
- removed the R1902 at (166.9, 37.5)
- removed the R1902 at (43.1, 62.5)
- removed the R1902 at (43.1, 92.5)
- removed the R1902 at (43.1, 122.5)
- removed the R1902 at (43.1, 152.5)
- removed the R1902 at (43.1, 182.5)
- removed the R1902 at (43.1, 212.5)
- removed the R1902 at (166.9, 217.5)
- removed the R1902 at (166.9, 187.5)
- removed the R1903 at (40.6, 12.1)
- removed the R1903 at (169.4, 177.9)
- removed the R1903 at (169.4, 147.9)
- removed the R1903 at (169.4, 117.9)
- removed the R1903 at (169.4, 87.9)
- removed the R1903 at (169.4, 57.9)
- removed the R1903 at (40.6, 42.1)
- removed the R1903 at (40.6, 72.1)
- removed the R1903 at (40.6, 102.1)
- removed the R1903 at (40.6, 132.1)
- removed the R1903 at (40.6, 162.1)
- removed the R1903 at (40.6, 192.1)
- removed the R1903 at (169.4, 237.9)
- removed the R1903 at (169.4, 207.9)
- removed the R1904 at (66.0, 12.1)
- removed the R1904 at (144.0, 177.9)
- removed the R1904 at (144.0, 147.9)
- removed the R1904 at (144.0, 117.9)
- removed the R1904 at (144.0, 87.9)
- removed the R1904 at (144.0, 57.9)
- removed the R1904 at (66.0, 42.1)
- removed the R1904 at (66.0, 72.1)
- removed the R1904 at (66.0, 102.1)
- removed the R1904 at (66.0, 132.1)
- removed the R1904 at (66.0, 162.1)
- removed the R1904 at (66.0, 192.1)
- removed the R1904 at (144.0, 237.9)
- removed the R1904 at (144.0, 207.9)
- removed the U1901 at (53.3, 22.3)
- removed the U1901 at (156.7, 167.7)
- removed the U1901 at (156.7, 137.7)
- removed the U1901 at (156.7, 107.7)
- removed the U1901 at (156.7, 77.7)
- removed the U1901 at (156.7, 47.7)
- removed the U1901 at (53.3, 52.3)
- removed the U1901 at (53.3, 82.3)
- removed the U1901 at (53.3, 112.3)
- removed the U1901 at (53.3, 142.3)
- removed the U1901 at (53.3, 172.3)
- removed the U1901 at (53.3, 202.3)
- removed the U1901 at (156.7, 227.7)
- removed the U1901 at (156.7, 197.7)
- added C1101: 100nF, Capacitor_THT:C_Disc_D8.0mm_W5.0mm_P5.00mm, F.Cu at (39.6, 203.7)
- added C1102: 100nF 6,3V, Capacitor_SMD:C_0201_0603Metric, F.Cu at (54.9, 210.0)
- added C1103: 100nF, Capacitor_THT:C_Disc_D8.0mm_W5.0mm_P5.00mm, F.Cu at (62.1, 203.6)
- added C1104: 1nF 25V, Capacitor_SMD:C_0201_0603Metric, B.Cu at (54.4, 210.3)
- added C1105: 33uF 35V, Capacitor_THT:CP_Radial_D5.0mm_P2.00mm, F.Cu at (21.5, 206.2)
- added C1106: 1nF 25V, Capacitor_SMD:C_0201_0603Metric, B.Cu at (55.4, 210.3)
- added C1107: 10nF 50V, Capacitor_SMD:C_0402_1005Metric, F.Cu at (44.4, 209.5)
- added C1108: 100nF 16V, Capacitor_SMD:C_0402_1005Metric, F.Cu at (43.4, 211.5)
- added C1201: 100nF, Capacitor_THT:C_Disc_D8.0mm_W5.0mm_P5.00mm, F.Cu at (39.6, 173.7)
- added C1202: 100nF 6,3V, Capacitor_SMD:C_0201_0603Metric, F.Cu at (54.9, 180.0)
- added C1203: 100nF, Capacitor_THT:C_Disc_D8.0mm_W5.0mm_P5.00mm, F.Cu at (62.1, 173.6)
- added C1204: 1nF 25V, Capacitor_SMD:C_0201_0603Metric, B.Cu at (54.4, 180.3)
- added C1205: 33uF 35V, Capacitor_THT:CP_Radial_D5.0mm_P2.00mm, F.Cu at (21.5, 176.2)
- added C1206: 1nF 25V, Capacitor_SMD:C_0201_0603Metric, B.Cu at (55.4, 180.3)
- added C1207: 10nF 50V, Capacitor_SMD:C_0402_1005Metric, F.Cu at (44.4, 179.5)
- added C1208: 100nF 16V, Capacitor_SMD:C_0402_1005Metric, F.Cu at (43.4, 181.5)
- added C1301: 100nF, Capacitor_THT:C_Disc_D8.0mm_W5.0mm_P5.00mm, F.Cu at (39.6, 143.7)
- added C1302: 100nF 6,3V, Capacitor_SMD:C_0201_0603Metric, F.Cu at (54.9, 150.0)
- added C1303: 100nF, Capacitor_THT:C_Disc_D8.0mm_W5.0mm_P5.00mm, F.Cu at (62.1, 143.6)
- added C1304: 1nF 25V, Capacitor_SMD:C_0201_0603Metric, B.Cu at (54.4, 150.3)
- added C1305: 33uF 35V, Capacitor_THT:CP_Radial_D5.0mm_P2.00mm, F.Cu at (21.5, 146.2)
- added C1306: 1nF 25V, Capacitor_SMD:C_0201_0603Metric, B.Cu at (55.4, 150.3)
- added C1307: 10nF 50V, Capacitor_SMD:C_0402_1005Metric, F.Cu at (44.4, 149.5)
- added C1308: 100nF 16V, Capacitor_SMD:C_0402_1005Metric, F.Cu at (43.4, 151.5)
- added C1401: 100nF, Capacitor_THT:C_Disc_D8.0mm_W5.0mm_P5.00mm, F.Cu at (39.6, 113.7)
- added C1402: 100nF 6,3V, Capacitor_SMD:C_0201_0603Metric, F.Cu at (54.9, 120.0)
- added C1403: 100nF, Capacitor_THT:C_Disc_D8.0mm_W5.0mm_P5.00mm, F.Cu at (62.1, 113.6)
- added C1404: 1nF 25V, Capacitor_SMD:C_0201_0603Metric, B.Cu at (54.4, 120.3)
- added C1405: 33uF 35V, Capacitor_THT:CP_Radial_D5.0mm_P2.00mm, F.Cu at (21.5, 116.2)
- added C1406: 1nF 25V, Capacitor_SMD:C_0201_0603Metric, B.Cu at (55.4, 120.3)
- added C1407: 10nF 50V, Capacitor_SMD:C_0402_1005Metric, F.Cu at (44.4, 119.5)
- added C1408: 100nF 16V, Capacitor_SMD:C_0402_1005Metric, F.Cu at (43.4, 121.5)
- added C1501: 100nF, Capacitor_THT:C_Disc_D8.0mm_W5.0mm_P5.00mm, F.Cu at (39.6, 83.7)
- added C1502: 100nF 6,3V, Capacitor_SMD:C_0201_0603Metric, F.Cu at (54.9, 90.0)
- added C1503: 100nF, Capacitor_THT:C_Disc_D8.0mm_W5.0mm_P5.00mm, F.Cu at (62.1, 83.6)
- added C1504: 1nF 25V, Capacitor_SMD:C_0201_0603Metric, B.Cu at (54.4, 90.3)
- added C1505: 33uF 35V, Capacitor_THT:CP_Radial_D5.0mm_P2.00mm, F.Cu at (21.5, 86.2)
- added C1506: 1nF 25V, Capacitor_SMD:C_0201_0603Metric, B.Cu at (55.4, 90.3)
- added C1507: 10nF 50V, Capacitor_SMD:C_0402_1005Metric, F.Cu at (44.4, 89.5)
- added C1508: 100nF 16V, Capacitor_SMD:C_0402_1005Metric, F.Cu at (43.4, 91.5)
- added C1601: 100nF, Capacitor_THT:C_Disc_D8.0mm_W5.0mm_P5.00mm, F.Cu at (39.6, 53.7)
- added C1602: 100nF 6,3V, Capacitor_SMD:C_0201_0603Metric, F.Cu at (54.9, 60.0)
- added C1603: 100nF, Capacitor_THT:C_Disc_D8.0mm_W5.0mm_P5.00mm, F.Cu at (62.1, 53.6)
- added C1604: 1nF 25V, Capacitor_SMD:C_0201_0603Metric, B.Cu at (54.4, 60.3)
- added C1605: 33uF 35V, Capacitor_THT:CP_Radial_D5.0mm_P2.00mm, F.Cu at (21.5, 56.1)
- added C1606: 1nF 25V, Capacitor_SMD:C_0201_0603Metric, B.Cu at (55.4, 60.3)
- added C1607: 10nF 50V, Capacitor_SMD:C_0402_1005Metric, F.Cu at (44.4, 59.5)
- added C1608: 100nF 16V, Capacitor_SMD:C_0402_1005Metric, F.Cu at (43.4, 61.5)
- added C1701: 100nF, Capacitor_THT:C_Disc_D8.0mm_W5.0mm_P5.00mm, F.Cu at (39.6, 23.7)
- added C1702: 100nF 6,3V, Capacitor_SMD:C_0201_0603Metric, F.Cu at (54.9, 30.0)
- added C1703: 100nF, Capacitor_THT:C_Disc_D8.0mm_W5.0mm_P5.00mm, F.Cu at (62.1, 23.6)
- added C1704: 1nF 25V, Capacitor_SMD:C_0201_0603Metric, B.Cu at (54.4, 30.3)
- added C1705: 33uF 35V, Capacitor_THT:CP_Radial_D5.0mm_P2.00mm, F.Cu at (21.5, 26.1)
- added C1706: 1nF 25V, Capacitor_SMD:C_0201_0603Metric, B.Cu at (55.4, 30.3)
- added C1707: 10nF 50V, Capacitor_SMD:C_0402_1005Metric, F.Cu at (44.4, 29.5)
- added C1708: 100nF 16V, Capacitor_SMD:C_0402_1005Metric, F.Cu at (43.4, 31.5)
- added C1801: 100nF, Capacitor_THT:C_Disc_D8.0mm_W5.0mm_P5.00mm, F.Cu at (160.4, 16.3)
- added C1802: 100nF 6,3V, Capacitor_SMD:C_0201_0603Metric, F.Cu at (145.1, 10.0)
- added C1803: 100nF, Capacitor_THT:C_Disc_D8.0mm_W5.0mm_P5.00mm, F.Cu at (137.9, 16.4)
- added C1804: 1nF 25V, Capacitor_SMD:C_0201_0603Metric, B.Cu at (145.6, 9.70)
- added C1805: 33uF 35V, Capacitor_THT:CP_Radial_D5.0mm_P2.00mm, F.Cu at (178.5, 13.8)
- added C1806: 1nF 25V, Capacitor_SMD:C_0201_0603Metric, B.Cu at (144.6, 9.68)
- added C1807: 10nF 50V, Capacitor_SMD:C_0402_1005Metric, F.Cu at (155.6, 10.5)
- added C1808: 100nF 16V, Capacitor_SMD:C_0402_1005Metric, F.Cu at (156.6, 8.50)
- added C2001: 100nF, Capacitor_THT:C_Disc_D8.0mm_W5.0mm_P5.00mm, F.Cu at (160.4, 76.3)
- added C2002: 100nF 6,3V, Capacitor_SMD:C_0201_0603Metric, F.Cu at (145.1, 70.0)
- added C2003: 100nF, Capacitor_THT:C_Disc_D8.0mm_W5.0mm_P5.00mm, F.Cu at (137.9, 76.4)
- added C2004: 1nF 25V, Capacitor_SMD:C_0201_0603Metric, B.Cu at (145.6, 69.7)
- added C2005: 33uF 35V, Capacitor_THT:CP_Radial_D5.0mm_P2.00mm, F.Cu at (178.5, 73.8)
- added C2006: 1nF 25V, Capacitor_SMD:C_0201_0603Metric, B.Cu at (144.6, 69.7)
- added C2007: 10nF 50V, Capacitor_SMD:C_0402_1005Metric, F.Cu at (155.6, 70.5)
- added C2008: 100nF 16V, Capacitor_SMD:C_0402_1005Metric, F.Cu at (156.6, 68.5)
- added C2101: 100nF, Capacitor_THT:C_Disc_D8.0mm_W5.0mm_P5.00mm, F.Cu at (160.4, 106.3)
- added C2102: 100nF 6,3V, Capacitor_SMD:C_0201_0603Metric, F.Cu at (145.1, 100.0)
- added C2103: 100nF, Capacitor_THT:C_Disc_D8.0mm_W5.0mm_P5.00mm, F.Cu at (137.9, 106.4)
- added C2104: 1nF 25V, Capacitor_SMD:C_0201_0603Metric, B.Cu at (145.6, 99.7)
- added C2105: 33uF 35V, Capacitor_THT:CP_Radial_D5.0mm_P2.00mm, F.Cu at (178.5, 103.8)
- added C2106: 1nF 25V, Capacitor_SMD:C_0201_0603Metric, B.Cu at (144.6, 99.7)
- added C2107: 10nF 50V, Capacitor_SMD:C_0402_1005Metric, F.Cu at (155.6, 100.5)
- added C2108: 100nF 16V, Capacitor_SMD:C_0402_1005Metric, F.Cu at (156.6, 98.5)
- added C2201: 100nF, Capacitor_THT:C_Disc_D8.0mm_W5.0mm_P5.00mm, F.Cu at (160.4, 136.3)
- added C2202: 100nF 6,3V, Capacitor_SMD:C_0201_0603Metric, F.Cu at (145.1, 130.0)
- added C2203: 100nF, Capacitor_THT:C_Disc_D8.0mm_W5.0mm_P5.00mm, F.Cu at (137.9, 136.4)
- added C2204: 1nF 25V, Capacitor_SMD:C_0201_0603Metric, B.Cu at (145.6, 129.7)
- added C2205: 33uF 35V, Capacitor_THT:CP_Radial_D5.0mm_P2.00mm, F.Cu at (178.5, 133.8)
- added C2206: 1nF 25V, Capacitor_SMD:C_0201_0603Metric, B.Cu at (144.6, 129.7)
- added C2207: 10nF 50V, Capacitor_SMD:C_0402_1005Metric, F.Cu at (155.6, 130.5)
- added C2208: 100nF 16V, Capacitor_SMD:C_0402_1005Metric, F.Cu at (156.6, 128.5)
- added C2301: 100nF, Capacitor_THT:C_Disc_D8.0mm_W5.0mm_P5.00mm, F.Cu at (160.4, 166.3)
- added C2302: 100nF 6,3V, Capacitor_SMD:C_0201_0603Metric, F.Cu at (145.1, 160.0)
- added C2303: 100nF, Capacitor_THT:C_Disc_D8.0mm_W5.0mm_P5.00mm, F.Cu at (137.9, 166.4)
- added C2304: 1nF 25V, Capacitor_SMD:C_0201_0603Metric, B.Cu at (145.6, 159.7)
- added C2305: 33uF 35V, Capacitor_THT:CP_Radial_D5.0mm_P2.00mm, F.Cu at (178.5, 163.8)
- added C2306: 1nF 25V, Capacitor_SMD:C_0201_0603Metric, B.Cu at (144.6, 159.7)
- added C2307: 10nF 50V, Capacitor_SMD:C_0402_1005Metric, F.Cu at (155.6, 160.5)
- added C2308: 100nF 16V, Capacitor_SMD:C_0402_1005Metric, F.Cu at (156.6, 158.5)
- added C2401: 100nF, Capacitor_THT:C_Disc_D8.0mm_W5.0mm_P5.00mm, F.Cu at (160.4, 196.3)
- added C2402: 100nF 6,3V, Capacitor_SMD:C_0201_0603Metric, F.Cu at (145.1, 190.0)
- added C2403: 100nF, Capacitor_THT:C_Disc_D8.0mm_W5.0mm_P5.00mm, F.Cu at (137.9, 196.4)
- added C2404: 1nF 25V, Capacitor_SMD:C_0201_0603Metric, B.Cu at (145.6, 189.7)
- added C2405: 33uF 35V, Capacitor_THT:CP_Radial_D5.0mm_P2.00mm, F.Cu at (178.5, 193.8)
- added C2406: 1nF 25V, Capacitor_SMD:C_0201_0603Metric, B.Cu at (144.6, 189.7)
- added C2407: 10nF 50V, Capacitor_SMD:C_0402_1005Metric, F.Cu at (155.6, 190.5)
- added C2408: 100nF 16V, Capacitor_SMD:C_0402_1005Metric, F.Cu at (156.6, 188.5)
- added C2501: 100nF, Capacitor_THT:C_Disc_D8.0mm_W5.0mm_P5.00mm, F.Cu at (160.4, 226.3)
- added C2502: 100nF 6,3V, Capacitor_SMD:C_0201_0603Metric, F.Cu at (145.1, 220.0)
- added C2503: 100nF, Capacitor_THT:C_Disc_D8.0mm_W5.0mm_P5.00mm, F.Cu at (137.9, 226.4)
- added C2504: 1nF 25V, Capacitor_SMD:C_0201_0603Metric, B.Cu at (145.6, 219.7)
- added C2505: 33uF 35V, Capacitor_THT:CP_Radial_D5.0mm_P2.00mm, F.Cu at (178.5, 223.8)
- added C2506: 1nF 25V, Capacitor_SMD:C_0201_0603Metric, B.Cu at (144.6, 219.7)
- added C2507: 10nF 50V, Capacitor_SMD:C_0402_1005Metric, F.Cu at (155.6, 220.5)
- added C2508: 100nF 16V, Capacitor_SMD:C_0402_1005Metric, F.Cu at (156.6, 218.5)
- added J1101: Screw_Terminal_01x04, Connector_Phoenix_MC_HighVoltage:PhoenixContact_MCV_1,5_4-G-5.08_1x04_P5.08mm_Vertical, F.Cu at (7.50, 207.5)
- added J1102: Screw_Terminal_01x04, Connector_Phoenix_MC_HighVoltage:PhoenixContact_MCV_1,5_4-G-5.08_1x04_P5.08mm_Vertical, F.Cu at (81.2, 192.2)
- added J1201: Screw_Terminal_01x04, Connector_Phoenix_MC_HighVoltage:PhoenixContact_MCV_1,5_4-G-5.08_1x04_P5.08mm_Vertical, F.Cu at (7.50, 177.5)
- added J1202: Screw_Terminal_01x04, Connector_Phoenix_MC_HighVoltage:PhoenixContact_MCV_1,5_4-G-5.08_1x04_P5.08mm_Vertical, F.Cu at (81.2, 162.2)
- added J1301: Screw_Terminal_01x04, Connector_Phoenix_MC_HighVoltage:PhoenixContact_MCV_1,5_4-G-5.08_1x04_P5.08mm_Vertical, F.Cu at (7.50, 147.5)
- added J1302: Screw_Terminal_01x04, Connector_Phoenix_MC_HighVoltage:PhoenixContact_MCV_1,5_4-G-5.08_1x04_P5.08mm_Vertical, F.Cu at (81.2, 132.2)
- added J1401: Screw_Terminal_01x04, Connector_Phoenix_MC_HighVoltage:PhoenixContact_MCV_1,5_4-G-5.08_1x04_P5.08mm_Vertical, F.Cu at (7.50, 117.5)
- added J1402: Screw_Terminal_01x04, Connector_Phoenix_MC_HighVoltage:PhoenixContact_MCV_1,5_4-G-5.08_1x04_P5.08mm_Vertical, F.Cu at (81.2, 102.2)
- added J1501: Screw_Terminal_01x04, Connector_Phoenix_MC_HighVoltage:PhoenixContact_MCV_1,5_4-G-5.08_1x04_P5.08mm_Vertical, F.Cu at (7.50, 87.5)
- added J1502: Screw_Terminal_01x04, Connector_Phoenix_MC_HighVoltage:PhoenixContact_MCV_1,5_4-G-5.08_1x04_P5.08mm_Vertical, F.Cu at (81.2, 72.2)
- added J1601: Screw_Terminal_01x04, Connector_Phoenix_MC_HighVoltage:PhoenixContact_MCV_1,5_4-G-5.08_1x04_P5.08mm_Vertical, F.Cu at (7.50, 57.5)
- added J1602: Screw_Terminal_01x04, Connector_Phoenix_MC_HighVoltage:PhoenixContact_MCV_1,5_4-G-5.08_1x04_P5.08mm_Vertical, F.Cu at (81.2, 42.2)
- added J1701: Screw_Terminal_01x04, Connector_Phoenix_MC_HighVoltage:PhoenixContact_MCV_1,5_4-G-5.08_1x04_P5.08mm_Vertical, F.Cu at (7.50, 27.5)
- added J1702: Screw_Terminal_01x04, Connector_Phoenix_MC_HighVoltage:PhoenixContact_MCV_1,5_4-G-5.08_1x04_P5.08mm_Vertical, F.Cu at (81.2, 12.2)
- added J1801: Screw_Terminal_01x04, Connector_Phoenix_MC_HighVoltage:PhoenixContact_MCV_1,5_4-G-5.08_1x04_P5.08mm_Vertical, F.Cu at (192.5, 12.5)
- added J1802: Screw_Terminal_01x04, Connector_Phoenix_MC_HighVoltage:PhoenixContact_MCV_1,5_4-G-5.08_1x04_P5.08mm_Vertical, F.Cu at (118.8, 27.8)
- added J2001: Screw_Terminal_01x04, Connector_Phoenix_MC_HighVoltage:PhoenixContact_MCV_1,5_4-G-5.08_1x04_P5.08mm_Vertical, F.Cu at (192.5, 72.5)
- added J2002: Screw_Terminal_01x04, Connector_Phoenix_MC_HighVoltage:PhoenixContact_MCV_1,5_4-G-5.08_1x04_P5.08mm_Vertical, F.Cu at (118.8, 87.8)
- added J2101: Screw_Terminal_01x04, Connector_Phoenix_MC_HighVoltage:PhoenixContact_MCV_1,5_4-G-5.08_1x04_P5.08mm_Vertical, F.Cu at (192.5, 102.5)
- added J2102: Screw_Terminal_01x04, Connector_Phoenix_MC_HighVoltage:PhoenixContact_MCV_1,5_4-G-5.08_1x04_P5.08mm_Vertical, F.Cu at (118.8, 117.8)
- added J2201: Screw_Terminal_01x04, Connector_Phoenix_MC_HighVoltage:PhoenixContact_MCV_1,5_4-G-5.08_1x04_P5.08mm_Vertical, F.Cu at (192.5, 132.5)
- added J2202: Screw_Terminal_01x04, Connector_Phoenix_MC_HighVoltage:PhoenixContact_MCV_1,5_4-G-5.08_1x04_P5.08mm_Vertical, F.Cu at (118.8, 147.8)
- added J2301: Screw_Terminal_01x04, Connector_Phoenix_MC_HighVoltage:PhoenixContact_MCV_1,5_4-G-5.08_1x04_P5.08mm_Vertical, F.Cu at (192.5, 162.5)
- added J2302: Screw_Terminal_01x04, Connector_Phoenix_MC_HighVoltage:PhoenixContact_MCV_1,5_4-G-5.08_1x04_P5.08mm_Vertical, F.Cu at (118.8, 177.8)
- added J2401: Screw_Terminal_01x04, Connector_Phoenix_MC_HighVoltage:PhoenixContact_MCV_1,5_4-G-5.08_1x04_P5.08mm_Vertical, F.Cu at (192.5, 192.5)
- added J2402: Screw_Terminal_01x04, Connector_Phoenix_MC_HighVoltage:PhoenixContact_MCV_1,5_4-G-5.08_1x04_P5.08mm_Vertical, F.Cu at (118.8, 207.8)
- added J2501: Screw_Terminal_01x04, Connector_Phoenix_MC_HighVoltage:PhoenixContact_MCV_1,5_4-G-5.08_1x04_P5.08mm_Vertical, F.Cu at (192.5, 222.5)
- added J2502: Screw_Terminal_01x04, Connector_Phoenix_MC_HighVoltage:PhoenixContact_MCV_1,5_4-G-5.08_1x04_P5.08mm_Vertical, F.Cu at (118.8, 237.8)
- added R1001: 0R5, Resistor_THT:R_Axial_DIN0411_L9.9mm_D3.6mm_P5.08mm_Vertical, F.Cu at (58.3, 240.0)
- added R1101: 0R5, Resistor_THT:R_Axial_DIN0411_L9.9mm_D3.6mm_P5.08mm_Vertical, F.Cu at (58.3, 210.0)
- added R1102: 0R5, Resistor_THT:R_Axial_DIN0411_L9.9mm_D3.6mm_P5.08mm_Vertical, F.Cu at (40.5, 210.0)
- added R1103: 0R5, Resistor_THT:R_Axial_DIN0411_L9.9mm_D3.6mm_P5.08mm_Vertical, F.Cu at (38.0, 189.6)
- added R1104: 0R5, Resistor_THT:R_Axial_DIN0411_L9.9mm_D3.6mm_P5.08mm_Vertical, F.Cu at (63.4, 189.6)
- added R1201: 0R5, Resistor_THT:R_Axial_DIN0411_L9.9mm_D3.6mm_P5.08mm_Vertical, F.Cu at (58.3, 180.0)
- added R1202: 0R5, Resistor_THT:R_Axial_DIN0411_L9.9mm_D3.6mm_P5.08mm_Vertical, F.Cu at (40.5, 180.0)
- added R1203: 0R5, Resistor_THT:R_Axial_DIN0411_L9.9mm_D3.6mm_P5.08mm_Vertical, F.Cu at (38.0, 159.6)
- added R1204: 0R5, Resistor_THT:R_Axial_DIN0411_L9.9mm_D3.6mm_P5.08mm_Vertical, F.Cu at (63.4, 159.6)
- added R1301: 0R5, Resistor_THT:R_Axial_DIN0411_L9.9mm_D3.6mm_P5.08mm_Vertical, F.Cu at (58.3, 150.0)
- added R1302: 0R5, Resistor_THT:R_Axial_DIN0411_L9.9mm_D3.6mm_P5.08mm_Vertical, F.Cu at (40.5, 150.0)
- added R1303: 0R5, Resistor_THT:R_Axial_DIN0411_L9.9mm_D3.6mm_P5.08mm_Vertical, F.Cu at (38.0, 129.6)
- added R1304: 0R5, Resistor_THT:R_Axial_DIN0411_L9.9mm_D3.6mm_P5.08mm_Vertical, F.Cu at (63.4, 129.6)
- added R1401: 0R5, Resistor_THT:R_Axial_DIN0411_L9.9mm_D3.6mm_P5.08mm_Vertical, F.Cu at (58.3, 120.0)
- added R1402: 0R5, Resistor_THT:R_Axial_DIN0411_L9.9mm_D3.6mm_P5.08mm_Vertical, F.Cu at (40.5, 120.0)
- added R1403: 0R5, Resistor_THT:R_Axial_DIN0411_L9.9mm_D3.6mm_P5.08mm_Vertical, F.Cu at (38.0, 99.6)
- added R1404: 0R5, Resistor_THT:R_Axial_DIN0411_L9.9mm_D3.6mm_P5.08mm_Vertical, F.Cu at (63.4, 99.6)
- added R1501: 0R5, Resistor_THT:R_Axial_DIN0411_L9.9mm_D3.6mm_P5.08mm_Vertical, F.Cu at (58.3, 90.0)
- added R1502: 0R5, Resistor_THT:R_Axial_DIN0411_L9.9mm_D3.6mm_P5.08mm_Vertical, F.Cu at (40.5, 90.0)
- added R1503: 0R5, Resistor_THT:R_Axial_DIN0411_L9.9mm_D3.6mm_P5.08mm_Vertical, F.Cu at (38.0, 69.6)
- added R1504: 0R5, Resistor_THT:R_Axial_DIN0411_L9.9mm_D3.6mm_P5.08mm_Vertical, F.Cu at (63.4, 69.6)
- added R1601: 0R5, Resistor_THT:R_Axial_DIN0411_L9.9mm_D3.6mm_P5.08mm_Vertical, F.Cu at (58.3, 60.0)
- added R1602: 0R5, Resistor_THT:R_Axial_DIN0411_L9.9mm_D3.6mm_P5.08mm_Vertical, F.Cu at (40.5, 60.0)
- added R1603: 0R5, Resistor_THT:R_Axial_DIN0411_L9.9mm_D3.6mm_P5.08mm_Vertical, F.Cu at (38.0, 39.6)
- added R1604: 0R5, Resistor_THT:R_Axial_DIN0411_L9.9mm_D3.6mm_P5.08mm_Vertical, F.Cu at (63.4, 39.6)
- added R1701: 0R5, Resistor_THT:R_Axial_DIN0411_L9.9mm_D3.6mm_P5.08mm_Vertical, F.Cu at (58.3, 30.0)
- added R1702: 0R5, Resistor_THT:R_Axial_DIN0411_L9.9mm_D3.6mm_P5.08mm_Vertical, F.Cu at (40.5, 30.0)
- added R1703: 0R5, Resistor_THT:R_Axial_DIN0411_L9.9mm_D3.6mm_P5.08mm_Vertical, F.Cu at (38.0, 9.64)
- added R1704: 0R5, Resistor_THT:R_Axial_DIN0411_L9.9mm_D3.6mm_P5.08mm_Vertical, F.Cu at (63.4, 9.64)
- added R1801: 0R5, Resistor_THT:R_Axial_DIN0411_L9.9mm_D3.6mm_P5.08mm_Vertical, F.Cu at (141.7, 10.0)
- added R1802: 0R5, Resistor_THT:R_Axial_DIN0411_L9.9mm_D3.6mm_P5.08mm_Vertical, F.Cu at (159.5, 10.0)
- added R1803: 0R5, Resistor_THT:R_Axial_DIN0411_L9.9mm_D3.6mm_P5.08mm_Vertical, F.Cu at (162.0, 30.4)
- added R1804: 0R5, Resistor_THT:R_Axial_DIN0411_L9.9mm_D3.6mm_P5.08mm_Vertical, F.Cu at (136.6, 30.4)
- added R2001: 0R5, Resistor_THT:R_Axial_DIN0411_L9.9mm_D3.6mm_P5.08mm_Vertical, F.Cu at (141.7, 70.0)
- added R2002: 0R5, Resistor_THT:R_Axial_DIN0411_L9.9mm_D3.6mm_P5.08mm_Vertical, F.Cu at (159.5, 70.0)
- added R2003: 0R5, Resistor_THT:R_Axial_DIN0411_L9.9mm_D3.6mm_P5.08mm_Vertical, F.Cu at (162.0, 90.4)
- added R2004: 0R5, Resistor_THT:R_Axial_DIN0411_L9.9mm_D3.6mm_P5.08mm_Vertical, F.Cu at (136.6, 90.4)
- added R2101: 0R5, Resistor_THT:R_Axial_DIN0411_L9.9mm_D3.6mm_P5.08mm_Vertical, F.Cu at (141.7, 100.0)
- added R2102: 0R5, Resistor_THT:R_Axial_DIN0411_L9.9mm_D3.6mm_P5.08mm_Vertical, F.Cu at (159.5, 100.0)
- added R2103: 0R5, Resistor_THT:R_Axial_DIN0411_L9.9mm_D3.6mm_P5.08mm_Vertical, F.Cu at (162.0, 120.4)
- added R2104: 0R5, Resistor_THT:R_Axial_DIN0411_L9.9mm_D3.6mm_P5.08mm_Vertical, F.Cu at (136.6, 120.4)
- added R2201: 0R5, Resistor_THT:R_Axial_DIN0411_L9.9mm_D3.6mm_P5.08mm_Vertical, F.Cu at (141.7, 130.0)
- added R2202: 0R5, Resistor_THT:R_Axial_DIN0411_L9.9mm_D3.6mm_P5.08mm_Vertical, F.Cu at (159.5, 130.0)
- added R2203: 0R5, Resistor_THT:R_Axial_DIN0411_L9.9mm_D3.6mm_P5.08mm_Vertical, F.Cu at (162.0, 150.4)
- added R2204: 0R5, Resistor_THT:R_Axial_DIN0411_L9.9mm_D3.6mm_P5.08mm_Vertical, F.Cu at (136.6, 150.4)
- added R2301: 0R5, Resistor_THT:R_Axial_DIN0411_L9.9mm_D3.6mm_P5.08mm_Vertical, F.Cu at (141.7, 160.0)
- added R2302: 0R5, Resistor_THT:R_Axial_DIN0411_L9.9mm_D3.6mm_P5.08mm_Vertical, F.Cu at (159.5, 160.0)
- added R2303: 0R5, Resistor_THT:R_Axial_DIN0411_L9.9mm_D3.6mm_P5.08mm_Vertical, F.Cu at (162.0, 180.4)
- added R2304: 0R5, Resistor_THT:R_Axial_DIN0411_L9.9mm_D3.6mm_P5.08mm_Vertical, F.Cu at (136.6, 180.4)
- added R2401: 0R5, Resistor_THT:R_Axial_DIN0411_L9.9mm_D3.6mm_P5.08mm_Vertical, F.Cu at (141.7, 190.0)
- added R2402: 0R5, Resistor_THT:R_Axial_DIN0411_L9.9mm_D3.6mm_P5.08mm_Vertical, F.Cu at (159.5, 190.0)
- added R2403: 0R5, Resistor_THT:R_Axial_DIN0411_L9.9mm_D3.6mm_P5.08mm_Vertical, F.Cu at (162.0, 210.4)
- added R2404: 0R5, Resistor_THT:R_Axial_DIN0411_L9.9mm_D3.6mm_P5.08mm_Vertical, F.Cu at (136.6, 210.4)
- added R2501: 0R5, Resistor_THT:R_Axial_DIN0411_L9.9mm_D3.6mm_P5.08mm_Vertical, F.Cu at (141.7, 220.0)
- added R2502: 0R5, Resistor_THT:R_Axial_DIN0411_L9.9mm_D3.6mm_P5.08mm_Vertical, F.Cu at (159.5, 220.0)
- added R2503: 0R5, Resistor_THT:R_Axial_DIN0411_L9.9mm_D3.6mm_P5.08mm_Vertical, F.Cu at (162.0, 240.4)
- added R2504: 0R5, Resistor_THT:R_Axial_DIN0411_L9.9mm_D3.6mm_P5.08mm_Vertical, F.Cu at (136.6, 240.4)
- added U1101: DRV8823, Package_SO:TSSOP-48_6.1x12.5mm_P0.5mm, F.Cu at (50.7, 199.8)
- added U1201: DRV8823, Package_SO:TSSOP-48_6.1x12.5mm_P0.5mm, F.Cu at (50.7, 169.8)
- added U1301: DRV8823, Package_SO:TSSOP-48_6.1x12.5mm_P0.5mm, F.Cu at (50.7, 139.8)
- added U1401: DRV8823, Package_SO:TSSOP-48_6.1x12.5mm_P0.5mm, F.Cu at (50.7, 109.8)
- added U1501: DRV8823, Package_SO:TSSOP-48_6.1x12.5mm_P0.5mm, F.Cu at (50.7, 79.8)
- added U1601: DRV8823, Package_SO:TSSOP-48_6.1x12.5mm_P0.5mm, F.Cu at (50.7, 49.8)
- added U1701: DRV8823, Package_SO:TSSOP-48_6.1x12.5mm_P0.5mm, F.Cu at (50.7, 19.8)
- added U1801: DRV8823, Package_SO:TSSOP-48_6.1x12.5mm_P0.5mm, F.Cu at (149.3, 20.2)
- added U2001: DRV8823, Package_SO:TSSOP-48_6.1x12.5mm_P0.5mm, F.Cu at (149.3, 80.2)
- added U2101: DRV8823, Package_SO:TSSOP-48_6.1x12.5mm_P0.5mm, F.Cu at (149.3, 110.2)
- added U2201: DRV8823, Package_SO:TSSOP-48_6.1x12.5mm_P0.5mm, F.Cu at (149.3, 140.2)
- added U2301: DRV8823, Package_SO:TSSOP-48_6.1x12.5mm_P0.5mm, F.Cu at (149.3, 170.2)
- added U2401: DRV8823, Package_SO:TSSOP-48_6.1x12.5mm_P0.5mm, F.Cu at (149.3, 200.2)
- added U2501: DRV8823, Package_SO:TSSOP-48_6.1x12.5mm_P0.5mm, F.Cu at (149.3, 230.2)
- moved C1901 33.4 mm to (160.3, 46.3)
- moved C1902 33.4 mm to (145.0, 40.0)
- moved C1903 33.4 mm to (137.8, 46.4)
- moved C1904 33.4 mm to (145.5, 39.7)
- moved C1905 33.4 mm to (178.4, 43.9)
- moved C1906 33.4 mm to (144.5, 39.7)
- moved C1907 33.4 mm to (155.5, 40.5)
- moved C1908 33.4 mm to (156.5, 38.5)
- moved J1901 33.4 mm to (192.4, 42.5)
- moved J1902 33.4 mm to (118.8, 57.8)
- moved R1901 33.4 mm to (141.6, 40.0)
- moved R1902 33.4 mm to (159.4, 40.0)
- moved R1903 33.4 mm to (161.9, 60.4)
- moved R1904 33.4 mm to (136.5, 60.4)
- moved U1901 33.4 mm to (149.2, 50.2)
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Connections:
- C1002 pad 1: Net-(C1902-Pad1) -> Net-(C1002-Pad1)
- C1007 pad 1: Net-(C1907-Pad1) -> Net-(C1007-Pad1)
- C1007 pad 2: Net-(C1907-Pad2) -> Net-(C1007-Pad2)
- C1008 pad 1: Net-(C1908-Pad1) -> Net-(C1008-Pad1)
- J1002 pad 1: /Motortreiber9/MC1 -> /Motortreiber0/MC1
- J1002 pad 2: /Motortreiber9/MC2 -> /Motortreiber0/MC2
- J1002 pad 3: /Motortreiber9/MD1 -> /Motortreiber0/MD1
- J1002 pad 4: /Motortreiber9/MD2 -> /Motortreiber0/MD2
- R1004 pad 2: /Motortreiber9/MCR -> /Motortreiber0/MCR
- U1001 pad 16: Net-(C1902-Pad1) -> Net-(C1002-Pad1)
- U1001 pad 19: Net-(U1901-Pad19) -> Net-(U1001-Pad19)
- U1001 pad 20: /Motortreiber9/MD2 -> /Motortreiber0/MD2
- U1001 pad 21: /Motortreiber9/MDR -> /Motortreiber0/MDR
- U1001 pad 22: /Motortreiber9/MD1 -> /Motortreiber0/MD1
- U1001 pad 25: /Motortreiber9/MC2 -> /Motortreiber0/MC2
- U1001 pad 26: /Motortreiber9/MCR -> /Motortreiber0/MCR
- U1001 pad 27: /Motortreiber9/MC1 -> /Motortreiber0/MC1
- U1001 pad 28: Net-(U1901-Pad28) -> Net-(U1001-Pad28)
- U1001 pad 29: Net-(U1901-Pad29) -> Net-(U1001-Pad29)
- U1001 pad 32: Net-(U1901-Pad32) -> Net-(U1001-Pad32)
- U1001 pad 40: Net-(U1901-Pad40) -> Net-(U1001-Pad40)
- U1001 pad 41: Net-(U1901-Pad41) -> Net-(U1001-Pad41)
- U1001 pad 44: Net-(U1901-Pad44) -> Net-(U1001-Pad44)
- U1001 pad 6: Net-(U1901-Pad6) -> Net-(U1001-Pad6)
- U1001 pad 7: Net-(C1907-Pad1) -> Net-(C1007-Pad1)
- U1001 pad 8: Net-(C1907-Pad2) -> Net-(C1007-Pad2)
- U1001 pad 9: Net-(C1908-Pad1) -> Net-(C1008-Pad1)
Routing:
- net /Motortreiber9/MA1: track 702.8 -> 46.9 mm, vias 15 -> 1
- net /Motortreiber9/MA2: track 654.9 -> 43.7 mm, vias 15 -> 1
- net /Motortreiber9/MB1: track 641.3 -> 42.8 mm, vias 15 -> 1
- net /Motortreiber9/MB2: track 597.4 -> 39.8 mm, vias 15 -> 1
- net /Motortreiber9/MD2: track 513.6 -> 32.1 mm, vias 16 -> 1
- net /Motortreiber9/MC1: track 501.1 -> 31.3 mm, vias 16 -> 1
- net /Motortreiber9/MD1: track 485.0 -> 30.3 mm, vias 16 -> 1
- net /Motortreiber9/MC2: track 434.1 -> 27.1 mm, vias 16 -> 1
- net /Strobe9: track 342.2 -> 19.5 mm, vias 15 -> 1
- net /Steuer4: track 560.5 -> 250.7 mm
- net /Steuer0: track 546.7 -> 241.8 mm
- net /Steuer1: track 530.5 -> 229.3 mm
- net /Steuer3: track 436.6 -> 176.1 mm
- net /Steuer2: track 419.6 -> 168.3 mm
- net /Steuer5: track 888.0 -> 654.9 mm
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Other:
- board size 210 x 290 mm -> 200 x 300 mm

Commit message: erster Treiber am Bus angeschlossen
Parts:
- added U501: ADUM3160, Package_SO:SOIC-16W_7.5x10.3mm_P1.27mm, F.Cu at (122.5, 272.5)
- added U502: ATxmega128C3-AU, Package_QFP:TQFP-64_14x14mm_P0.8mm, F.Cu at (92.1, 270.7)
Routing:
- net /Steuer6: track 688.4 -> 1006.4 mm, vias 16 -> 19
- net /Steuer5: track 654.9 -> 972.7 mm, vias 16 -> 19
- net /Steuer3: track 176.1 -> 480.5 mm, vias 16 -> 19
- net /Steuer4: track 250.7 -> 554.8 mm, vias 16 -> 19
- net /Steuer1: track 229.3 -> 533.3 mm, vias 16 -> 19
- net /Steuer2: track 168.3 -> 471.9 mm, vias 16 -> 19
- net /Steuer0: track 241.8 -> 545.2 mm, vias 16 -> 19
- net /Strobe9: track 19.5 -> 318.4 mm, vias 1 -> 2
- net /Strobe8: track 10.6 -> 289.4 mm, vias 1 -> 2

Commit message: erster Treiber neu am Bus angebunden
Routing:
- net /Strobe9: track 318.4 -> 333.3 mm
- net /Steuer0: track 545.2 -> 550.7 mm
- net /Steuer3: track 480.5 -> 485.8 mm
- net /Steuer2: track 471.9 -> 477.0 mm
- net /Steuer5: track 972.7 -> 977.6 mm
- net /Steuer1: track 533.3 -> 537.2 mm
- net /Steuer6: track 1006.4 -> 1010.0 mm
- net /Steuer4: track 554.8 -> 558.0 mm

Commit message: Mittlerer Bus verschoben Fehler in Steuer2
Parts:
- moved U501 103.9 mm to (19.5, 259.0)
- moved U502 4.50 mm to (96.6, 270.7)
Routing:
- net /Steuer2: track 477.0 -> 297.5 mm
- net /Strobe5: track 2.57 -> 124.0 mm, vias 1 -> 2
- net /Strobe7: track 10.6 -> 72.4 mm, vias 1 -> 2
- net /Strobe6: track 10.6 -> 72.0 mm, vias 1 -> 2
- net /Strobe4: track 10.6 -> 70.9 mm, vias 1 -> 2
- net /Strobe3: track 10.6 -> 70.6 mm, vias 1 -> 2
- net /Steuer5: track 977.6 -> 1030.6 mm, vias 19 -> 21
- net /Steuer6: track 1010.0 -> 1060.9 mm, vias 19 -> 21
- net /Strobe2: track 10.6 -> 60.0 mm, vias 1 -> 2
- net /Strobe1: track 10.6 -> 58.4 mm, vias 1 -> 2
- net /Strobe0: track 10.6 -> 57.1 mm, vias 1 -> 2
- net /Steuer4: track 558.0 -> 568.5 mm
- net /Steuer1: track 537.2 -> 546.2 mm
- net /Steuer0: track 550.7 -> 558.2 mm
- net /Steuer3: track 485.8 -> 490.7 mm
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
Commit message: weitere Motortreiber am Bus angebunden
Parts:
- moved U501 33.1 mm to (17.5, 292.0)
- moved U502 8.50 mm to (96.6, 279.2)
- moved J2501 6.00 mm to (186.5, 222.5)
- moved C1504 1.75 mm to (53.0, 91.3), turned to 270 degrees
- moved C1904 1.50 mm to (147.0, 39.7)
- moved C1604 1.43 mm to (53.0, 60.5), turned to 270 degrees
- moved C2004 1.43 mm to (147.0, 69.8), turned to 90 degrees
- moved C2104 1.43 mm to (147.0, 99.8), turned to 90 degrees
- moved C1506 1.00 mm to (55.5, 91.3), turned to 270 degrees
- moved C1804 0.93 mm to (146.5, 9.82), turned to 90 degrees
- moved C1704 0.92 mm to (53.5, 30.3), turned to 270 degrees
- moved C1606 0.37 mm to (55.5, 60.7), turned to 270 degrees
- moved C1706 0.20 mm to (55.5, 30.5), turned to 270 degrees
- moved C2106 0.16 mm to (144.5, 99.8), turned to 90 degrees
- turned C1806 to 90 degrees
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Routing:
- net /Steuer2: track 297.5 -> 770.6 mm, vias 19 -> 31
- net +28V: track 1308.6 -> 1645.3 mm
- net /Steuer0: track 558.2 -> 867.7 mm, vias 19 -> 31
- net /Steuer4: track 568.5 -> 876.1 mm, vias 19 -> 28
- net /Steuer1: track 546.2 -> 853.7 mm, vias 19 -> 31
- net /Strobe7: track 72.4 -> 369.9 mm
- net /Steuer3: track 490.7 -> 780.0 mm, vias 19 -> 29
- net /Strobe10: track 10.6 -> 294.6 mm, vias 1 -> 2
- net /Strobe6: track 72.0 -> 337.1 mm
- net /Strobe4: track 70.9 -> 284.6 mm
- net /Strobe11: track 10.6 -> 203.8 mm, vias 1 -> 2
- net /Strobe5: track 124.0 -> 304.9 mm
- net /Strobe12: track 10.6 -> 173.1 mm, vias 1 -> 2
- net /Strobe13: track 10.6 -> 150.6 mm, vias 1 -> 2
- net /Strobe3: track 70.6 -> 206.1 mm
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Other:
- net class USB added: clearance 0.2, trace_width 0.25, via_dia 0.8, via_drill 0.4
