File: Hardware/Motortreiber002/Motorteiber002.kicad_pcb (KiCad board)
At the start: 2 copper layers, 200 x 300 mm, 242 parts, among them J1001 Screw_Terminal_01x04, J1002 Screw_Terminal_01x04, J1101 Screw_Terminal_01x04, J1102 Screw_Terminal_01x04, J1201 Screw_Terminal_01x04, J1202 Screw_Terminal_01x04, J1301 Screw_Terminal_01x04, J1302 Screw_Terminal_01x04, J1401 Screw_Terminal_01x04, J1402 Screw_Terminal_01x04, J1501 Screw_Terminal_01x04, J1502 Screw_Terminal_01x04, J1601 Screw_Terminal_01x04, J1602 Screw_Terminal_01x04, J1701 Screw_Terminal_01x04, J1702 Screw_Terminal_01x04, J1801 Screw_Terminal_01x04, J1802 Screw_Terminal_01x04, J1901 Screw_Terminal_01x04, J1902 Screw_Terminal_01x04, J2001 Screw_Terminal_01x04, J2002 Screw_Terminal_01x04, J2101 Screw_Terminal_01x04, J2102 Screw_Terminal_01x04, J2201 Screw_Terminal_01x04, J2202 Screw_Terminal_01x04, J2301 Screw_Terminal_01x04, J2302 Screw_Terminal_01x04, J2401 Screw_Terminal_01x04, J2402 Screw_Terminal_01x04, J2501 Screw_Terminal_01x04, J2502 Screw_Terminal_01x04, U1001 DRV8823, U1101 DRV8823, U1201 DRV8823, U1301 DRV8823, U1401 DRV8823, U1501 DRV8823, U1601 DRV8823, U1701 DRV8823, U1801 DRV8823, U1901 DRV8823, U2001 DRV8823, U2101 DRV8823, U2201 DRV8823, U2301 DRV8823, U2401 DRV8823, U2501 DRV8823, U501 ADUM3160, U502 ATxmega128C3-AU

Commit message: Motortreiber letzte Aenderungen
Parts:
- removed C1801, C1803, C1901, C1903, C2001, C2003, C2101, C2103, C2201, C2203, C2301, C2303, C2401, C2403, C2501, C2503: 100nF, Capacitor_THT:C_Disc_D8.0mm_W5.0mm_P5.00mm
- removed C1802, C1902, C2002, C2102, C2202, C2302, C2402, C2502: 100nF 6,3V, Capacitor_SMD:C_0201_0603Metric
- removed C1804, C1806, C1904, C1906, C2004, C2006, C2104, C2106, C2204, C2206, C2304, C2306, C2404, C2406, C2504, C2506: 1nF 25V, Capacitor_SMD:C_0201_0603Metric
- removed C1805, C1905, C2005, C2105, C2205, C2305, C2405, C2505: 33uF 35V, Capacitor_THT:CP_Radial_D5.0mm_P2.00mm
- removed C1807, C1907, C2007, C2107, C2207, C2307, C2407, C2507: 10nF 50V, Capacitor_SMD:C_0402_1005Metric
- removed C1808, C1908, C2008, C2108, C2208, C2308, C2408, C2508: 100nF 16V, Capacitor_SMD:C_0402_1005Metric
- removed J1801, J1802, J1901, J1902, J2001, J2002, J2101, J2102, J2201, J2202, J2301, J2302, J2401, J2402, J2501, J2502: Screw_Terminal_01x04, Connector_Phoenix_MC_HighVoltage:PhoenixContact_MCV_1,5_4-G-5.08_1x04_P5.08mm_Vertical
- removed R1801, R1802, R1803, R1804, R1901, R1902, R1903, R1904, R2001, R2002, R2003, R2004, R2101, R2102, R2103, R2104, R2201, R2202, R2203, R2204, R2301, R2302, R2303, R2304, R2401, R2402, R2403, R2404, R2501, R2502, R2503, R2504: 0R5, Resistor_THT:R_Axial_DIN0411_L9.9mm_D3.6mm_P5.08mm_Vertical
- removed U1801, U1901, U2001, U2101, U2201, U2301, U2401, U2501: DRV8823, Package_SO:TSSOP-48_6.1x12.5mm_P0.5mm
- added C301: 100nF, Capacitor_THT:C_Disc_D8.0mm_W5.0mm_P5.00mm, F.Cu at (37.6, 10.8)
- added C302: 100nF, Capacitor_THT:C_Disc_D8.0mm_W5.0mm_P5.00mm, F.Cu at (37.6, 24.8)
- added C303: 100nF 6,3V, Capacitor_SMD:C_0201_0603Metric, F.Cu at (44.0, 19.7)
- added C304: 1nF 25V, Capacitor_SMD:C_0201_0603Metric, F.Cu at (42.7, 19.7)
- added C305: 33uF 35V, Capacitor_THT:CP_Radial_D5.0mm_P2.00mm, F.Cu at (31.5, 10.5)
- added C306: 1nF 25V, Capacitor_SMD:C_0201_0603Metric, F.Cu at (41.4, 19.7)
- added C307: 10nF 50V, Capacitor_SMD:C_0402_1005Metric, F.Cu at (45.2, 14.6)
- added C308: 100nF 16V, Capacitor_SMD:C_0402_1005Metric, F.Cu at (44.0, 14.6)
- added C401: 100nF, Capacitor_THT:C_Disc_D8.0mm_W5.0mm_P5.00mm, F.Cu at (37.6, 46.8)
- added C402: 100nF, Capacitor_THT:C_Disc_D8.0mm_W5.0mm_P5.00mm, F.Cu at (37.6, 60.8)
- added C403: 100nF 6,3V, Capacitor_SMD:C_0201_0603Metric, F.Cu at (44.0, 55.7)
- added C404: 1nF 25V, Capacitor_SMD:C_0201_0603Metric, F.Cu at (42.7, 55.7)
- added C405: 33uF 35V, Capacitor_THT:CP_Radial_D5.0mm_P2.00mm, F.Cu at (31.5, 46.5)
- added C406: 1nF 25V, Capacitor_SMD:C_0201_0603Metric, F.Cu at (41.4, 55.7)
- added C407: 10nF 50V, Capacitor_SMD:C_0402_1005Metric, F.Cu at (45.2, 50.6)
- added C408: 100nF 16V, Capacitor_SMD:C_0402_1005Metric, F.Cu at (44.0, 50.6)
- added C501: 100nF, Capacitor_SMD:C_0603_1608Metric_Pad1.05x0.95mm_HandSolder, F.Cu at (139.5, 257.5)
- added C502: 100nF, Capacitor_SMD:C_0603_1608Metric_Pad1.05x0.95mm_HandSolder, F.Cu at (120.0, 252.0)
- added C503: 100nF, Capacitor_SMD:C_0603_1608Metric_Pad1.05x0.95mm_HandSolder, F.Cu at (132.5, 252.5)
- added C504: 100nF, Capacitor_SMD:C_0603_1608Metric_Pad1.05x0.95mm_HandSolder, F.Cu at (138.0, 270.0)
- added C505: 100nF, Capacitor_SMD:C_0603_1608Metric_Pad1.05x0.95mm_HandSolder, F.Cu at (121.0, 275.5)
- added C506: 100nF, Capacitor_SMD:C_0603_1608Metric_Pad1.05x0.95mm_HandSolder, F.Cu at (116.5, 257.5)
- added C507: 100nF, Capacitor_SMD:C_0603_1608Metric_Pad1.05x0.95mm_HandSolder, F.Cu at (115.5, 270.0)
- added C601: 100nF, Capacitor_THT:C_Disc_D8.0mm_W5.0mm_P5.00mm, F.Cu at (37.6, 82.8)
- added C602: 100nF, Capacitor_THT:C_Disc_D8.0mm_W5.0mm_P5.00mm, F.Cu at (37.6, 96.8)
- added C603: 100nF 6,3V, Capacitor_SMD:C_0201_0603Metric, F.Cu at (44.0, 91.7)
- added C604: 1nF 25V, Capacitor_SMD:C_0201_0603Metric, F.Cu at (42.7, 91.7)
- added C605: 33uF 35V, Capacitor_THT:CP_Radial_D5.0mm_P2.00mm, F.Cu at (31.5, 82.5)
- added C606: 1nF 25V, Capacitor_SMD:C_0201_0603Metric, F.Cu at (41.4, 91.7)
- added C607: 10nF 50V, Capacitor_SMD:C_0402_1005Metric, F.Cu at (45.2, 86.6)
- added C608: 100nF 16V, Capacitor_SMD:C_0402_1005Metric, F.Cu at (44.0, 86.6)
- added C701: 100nF, Capacitor_THT:C_Disc_D8.0mm_W5.0mm_P5.00mm, F.Cu at (37.6, 118.8)
- added C702: 100nF, Capacitor_THT:C_Disc_D8.0mm_W5.0mm_P5.00mm, F.Cu at (37.6, 132.8)
- added C703: 100nF 6,3V, Capacitor_SMD:C_0201_0603Metric, F.Cu at (44.0, 127.7)
- added C704: 1nF 25V, Capacitor_SMD:C_0201_0603Metric, F.Cu at (42.7, 127.7)
- added C705: 33uF 35V, Capacitor_THT:CP_Radial_D5.0mm_P2.00mm, F.Cu at (31.5, 118.5)
- added C706: 1nF 25V, Capacitor_SMD:C_0201_0603Metric, F.Cu at (41.4, 127.7)
- added C707: 10nF 50V, Capacitor_SMD:C_0402_1005Metric, F.Cu at (45.2, 122.6)
- added C708: 100nF 16V, Capacitor_SMD:C_0402_1005Metric, F.Cu at (44.0, 122.6)
- added C801: 100nF, Capacitor_THT:C_Disc_D8.0mm_W5.0mm_P5.00mm, F.Cu at (37.6, 154.8)
- added C802: 100nF, Capacitor_THT:C_Disc_D8.0mm_W5.0mm_P5.00mm, F.Cu at (37.6, 168.8)
- added C803: 100nF 6,3V, Capacitor_SMD:C_0201_0603Metric, F.Cu at (44.0, 163.7)
- added C804: 1nF 25V, Capacitor_SMD:C_0201_0603Metric, F.Cu at (42.7, 163.7)
- added C805: 33uF 35V, Capacitor_THT:CP_Radial_D5.0mm_P2.00mm, F.Cu at (31.5, 154.5)
- added C806: 1nF 25V, Capacitor_SMD:C_0201_0603Metric, F.Cu at (41.4, 163.7)
- added C807: 10nF 50V, Capacitor_SMD:C_0402_1005Metric, F.Cu at (45.2, 158.6)
- added C808: 100nF 16V, Capacitor_SMD:C_0402_1005Metric, F.Cu at (44.0, 158.6)
- added C901: 100nF, Capacitor_THT:C_Disc_D8.0mm_W5.0mm_P5.00mm, F.Cu at (37.6, 190.8)
- added C902: 100nF, Capacitor_THT:C_Disc_D8.0mm_W5.0mm_P5.00mm, F.Cu at (37.6, 204.8)
- added C903: 100nF 6,3V, Capacitor_SMD:C_0201_0603Metric, F.Cu at (44.0, 199.7)
- added C904: 1nF 25V, Capacitor_SMD:C_0201_0603Metric, F.Cu at (42.7, 199.7)
- added C905: 33uF 35V, Capacitor_THT:CP_Radial_D5.0mm_P2.00mm, F.Cu at (31.5, 190.5)
- added C906: 1nF 25V, Capacitor_SMD:C_0201_0603Metric, F.Cu at (41.4, 199.7)
- added C907: 10nF 50V, Capacitor_SMD:C_0402_1005Metric, F.Cu at (45.2, 194.6)
- added C908: 100nF 16V, Capacitor_SMD:C_0402_1005Metric, F.Cu at (44.0, 194.6)
- added J301: Screw_Terminal_01x08, TerminalBlock_Phoenix:TerminalBlock_Phoenix_PT-1,5-8-3.5-H_1x08_P3.50mm_Horizontal, F.Cu at (5.50, 31.0)
- added J302: Conn_01x10_Male, Connector_PinHeader_1.00mm:PinHeader_1x10_P1.00mm_Vertical, F.Cu at (81.5, 25.0)
- added J401: Screw_Terminal_01x08, TerminalBlock_Phoenix:TerminalBlock_Phoenix_PT-1,5-8-3.5-H_1x08_P3.50mm_Horizontal, F.Cu at (5.50, 67.0)
- added J402: Conn_01x10_Male, Connector_PinHeader_1.00mm:PinHeader_1x10_P1.00mm_Vertical, F.Cu at (81.5, 61.0)
- added J601: Screw_Terminal_01x08, TerminalBlock_Phoenix:TerminalBlock_Phoenix_PT-1,5-8-3.5-H_1x08_P3.50mm_Horizontal, F.Cu at (5.50, 103.0)
- added J602: Conn_01x10_Male, Connector_PinHeader_1.00mm:PinHeader_1x10_P1.00mm_Vertical, F.Cu at (81.5, 97.0)
- added J701: Screw_Terminal_01x08, TerminalBlock_Phoenix:TerminalBlock_Phoenix_PT-1,5-8-3.5-H_1x08_P3.50mm_Horizontal, F.Cu at (5.50, 139.0)
- added J702: Conn_01x10_Male, Connector_PinHeader_1.00mm:PinHeader_1x10_P1.00mm_Vertical, F.Cu at (81.5, 133.0)
- added J801: Screw_Terminal_01x08, TerminalBlock_Phoenix:TerminalBlock_Phoenix_PT-1,5-8-3.5-H_1x08_P3.50mm_Horizontal, F.Cu at (5.50, 175.0)
- added J802: Conn_01x10_Male, Connector_PinHeader_1.00mm:PinHeader_1x10_P1.00mm_Vertical, F.Cu at (81.5, 169.0)
- added J901: Screw_Terminal_01x08, TerminalBlock_Phoenix:TerminalBlock_Phoenix_PT-1,5-8-3.5-H_1x08_P3.50mm_Horizontal, F.Cu at (5.50, 211.0)
- added J902: Conn_01x10_Male, Connector_PinHeader_1.00mm:PinHeader_1x10_P1.00mm_Vertical, F.Cu at (81.5, 205.0)
- added R1005: R, Resistor_THT:R_Axial_DIN0204_L3.6mm_D1.6mm_P2.54mm_Vertical, F.Cu at (69.5, 244.5)
- added R1006: 1, Resistor_THT:R_Axial_DIN0204_L3.6mm_D1.6mm_P2.54mm_Vertical, F.Cu at (72.5, 242.0)
- added R1007: 0R5, Resistor_THT:R_Axial_DIN0411_L9.9mm_D3.6mm_P5.08mm_Vertical, F.Cu at (27.4, 237.7)
- added R1008: 0R5, Resistor_THT:R_Axial_DIN0411_L9.9mm_D3.6mm_P5.08mm_Vertical, F.Cu at (27.4, 232.6)
- added R1009: 0R5, Resistor_THT:R_Axial_DIN0411_L9.9mm_D3.6mm_P5.08mm_Vertical, F.Cu at (59.0, 219.5)
- added R1010: 0R5, Resistor_THT:R_Axial_DIN0411_L9.9mm_D3.6mm_P5.08mm_Vertical, F.Cu at (57.5, 249.0)
- added R1105: R, Resistor_THT:R_Axial_DIN0204_L3.6mm_D1.6mm_P2.54mm_Vertical, F.Cu at (129.5, 225.0)
- added R1106: 1, Resistor_THT:R_Axial_DIN0204_L3.6mm_D1.6mm_P2.54mm_Vertical, F.Cu at (126.5, 227.5)
- added R1107: 0R5, Resistor_THT:R_Axial_DIN0411_L9.9mm_D3.6mm_P5.08mm_Vertical, F.Cu at (171.6, 231.8)
- added R1108: 0R5, Resistor_THT:R_Axial_DIN0411_L9.9mm_D3.6mm_P5.08mm_Vertical, F.Cu at (171.6, 236.9)
- added R1109: 0R5, Resistor_THT:R_Axial_DIN0411_L9.9mm_D3.6mm_P5.08mm_Vertical, F.Cu at (140.0, 250.0)
- added R1110: 0R5, Resistor_THT:R_Axial_DIN0411_L9.9mm_D3.6mm_P5.08mm_Vertical, F.Cu at (141.5, 220.5)
- added R1205: R, Resistor_THT:R_Axial_DIN0204_L3.6mm_D1.6mm_P2.54mm_Vertical, F.Cu at (129.5, 189.0)
- added R1206: 1, Resistor_THT:R_Axial_DIN0204_L3.6mm_D1.6mm_P2.54mm_Vertical, F.Cu at (126.5, 191.5)
- added R1207: 0R5, Resistor_THT:R_Axial_DIN0411_L9.9mm_D3.6mm_P5.08mm_Vertical, F.Cu at (171.6, 195.8)
- added R1208: 0R5, Resistor_THT:R_Axial_DIN0411_L9.9mm_D3.6mm_P5.08mm_Vertical, F.Cu at (171.6, 200.9)
- added R1209: 0R5, Resistor_THT:R_Axial_DIN0411_L9.9mm_D3.6mm_P5.08mm_Vertical, F.Cu at (140.0, 214.0)
- added R1210: 0R5, Resistor_THT:R_Axial_DIN0411_L9.9mm_D3.6mm_P5.08mm_Vertical, F.Cu at (141.5, 184.5)
- added R1305: R, Resistor_THT:R_Axial_DIN0204_L3.6mm_D1.6mm_P2.54mm_Vertical, F.Cu at (129.5, 153.0)
- added R1306: 1, Resistor_THT:R_Axial_DIN0204_L3.6mm_D1.6mm_P2.54mm_Vertical, F.Cu at (126.5, 155.5)
- added R1307: 0R5, Resistor_THT:R_Axial_DIN0411_L9.9mm_D3.6mm_P5.08mm_Vertical, F.Cu at (171.6, 159.8)
- added R1308: 0R5, Resistor_THT:R_Axial_DIN0411_L9.9mm_D3.6mm_P5.08mm_Vertical, F.Cu at (171.6, 164.9)
- added R1309: 0R5, Resistor_THT:R_Axial_DIN0411_L9.9mm_D3.6mm_P5.08mm_Vertical, F.Cu at (140.0, 178.0)
- added R1310: 0R5, Resistor_THT:R_Axial_DIN0411_L9.9mm_D3.6mm_P5.08mm_Vertical, F.Cu at (141.5, 148.5)
- added R1405: R, Resistor_THT:R_Axial_DIN0204_L3.6mm_D1.6mm_P2.54mm_Vertical, F.Cu at (129.5, 117.0)
- added R1406: 1, Resistor_THT:R_Axial_DIN0204_L3.6mm_D1.6mm_P2.54mm_Vertical, F.Cu at (126.5, 119.5)
- added R1407: 0R5, Resistor_THT:R_Axial_DIN0411_L9.9mm_D3.6mm_P5.08mm_Vertical, F.Cu at (171.6, 123.8)
- added R1408: 0R5, Resistor_THT:R_Axial_DIN0411_L9.9mm_D3.6mm_P5.08mm_Vertical, F.Cu at (171.6, 128.9)
- added R1409: 0R5, Resistor_THT:R_Axial_DIN0411_L9.9mm_D3.6mm_P5.08mm_Vertical, F.Cu at (140.0, 142.0)
- added R1410: 0R5, Resistor_THT:R_Axial_DIN0411_L9.9mm_D3.6mm_P5.08mm_Vertical, F.Cu at (141.5, 112.5)
- added R1505: R, Resistor_THT:R_Axial_DIN0204_L3.6mm_D1.6mm_P2.54mm_Vertical, F.Cu at (129.5, 81.0)
- added R1506: 1, Resistor_THT:R_Axial_DIN0204_L3.6mm_D1.6mm_P2.54mm_Vertical, F.Cu at (126.5, 83.5)
- added R1507: 0R5, Resistor_THT:R_Axial_DIN0411_L9.9mm_D3.6mm_P5.08mm_Vertical, F.Cu at (171.6, 87.8)
- added R1508: 0R5, Resistor_THT:R_Axial_DIN0411_L9.9mm_D3.6mm_P5.08mm_Vertical, F.Cu at (171.6, 92.9)
- added R1509: 0R5, Resistor_THT:R_Axial_DIN0411_L9.9mm_D3.6mm_P5.08mm_Vertical, F.Cu at (140.0, 106.0)
- added R1510: 0R5, Resistor_THT:R_Axial_DIN0411_L9.9mm_D3.6mm_P5.08mm_Vertical, F.Cu at (141.5, 76.5)
- added R1605: R, Resistor_THT:R_Axial_DIN0204_L3.6mm_D1.6mm_P2.54mm_Vertical, F.Cu at (129.5, 45.0)
- added R1606: 1, Resistor_THT:R_Axial_DIN0204_L3.6mm_D1.6mm_P2.54mm_Vertical, F.Cu at (126.5, 47.5)
- added R1607: 0R5, Resistor_THT:R_Axial_DIN0411_L9.9mm_D3.6mm_P5.08mm_Vertical, F.Cu at (171.6, 51.8)
- added R1608: 0R5, Resistor_THT:R_Axial_DIN0411_L9.9mm_D3.6mm_P5.08mm_Vertical, F.Cu at (171.6, 56.9)
- added R1609: 0R5, Resistor_THT:R_Axial_DIN0411_L9.9mm_D3.6mm_P5.08mm_Vertical, F.Cu at (140.0, 70.0)
- added R1610: 0R5, Resistor_THT:R_Axial_DIN0411_L9.9mm_D3.6mm_P5.08mm_Vertical, F.Cu at (141.5, 40.5)
- added R1705: R, Resistor_THT:R_Axial_DIN0204_L3.6mm_D1.6mm_P2.54mm_Vertical, F.Cu at (129.5, 9.00)
- added R1706: 1, Resistor_THT:R_Axial_DIN0204_L3.6mm_D1.6mm_P2.54mm_Vertical, F.Cu at (126.5, 11.5)
- added R1707: 0R5, Resistor_THT:R_Axial_DIN0411_L9.9mm_D3.6mm_P5.08mm_Vertical, F.Cu at (171.6, 15.8)
- added R1708: 0R5, Resistor_THT:R_Axial_DIN0411_L9.9mm_D3.6mm_P5.08mm_Vertical, F.Cu at (171.6, 20.9)
- added R1709: 0R5, Resistor_THT:R_Axial_DIN0411_L9.9mm_D3.6mm_P5.08mm_Vertical, F.Cu at (140.0, 34.0)
- added R1710: 0R5, Resistor_THT:R_Axial_DIN0411_L9.9mm_D3.6mm_P5.08mm_Vertical, F.Cu at (141.5, 4.50)
- added R301: R, Resistor_THT:R_Axial_DIN0204_L3.6mm_D1.6mm_P2.54mm_Vertical, F.Cu at (66.5, 34.0)
- added R302: R, Resistor_THT:R_Axial_DIN0204_L3.6mm_D1.6mm_P2.54mm_Vertical, F.Cu at (69.5, 31.5)
- added R303: 1, Resistor_THT:R_Axial_DIN0204_L3.6mm_D1.6mm_P2.54mm_Vertical, F.Cu at (72.5, 34.0)
- added R304: R, Resistor_THT:R_Axial_DIN0204_L3.6mm_D1.6mm_P2.54mm_Vertical, F.Cu at (66.5, 26.0)
- added R305: R, Resistor_THT:R_Axial_DIN0204_L3.6mm_D1.6mm_P2.54mm_Vertical, F.Cu at (69.5, 28.5)
- added R306: 1, Resistor_THT:R_Axial_DIN0204_L3.6mm_D1.6mm_P2.54mm_Vertical, F.Cu at (72.5, 26.0)
- added R307: 0R5, Resistor_THT:R_Axial_DIN0411_L9.9mm_D3.6mm_P5.08mm_Vertical, F.Cu at (27.4, 21.7)
- added R308: 0R5, Resistor_THT:R_Axial_DIN0411_L9.9mm_D3.6mm_P5.08mm_Vertical, F.Cu at (27.4, 16.6)
- added R309: 0R5, Resistor_THT:R_Axial_DIN0411_L9.9mm_D3.6mm_P5.08mm_Vertical, F.Cu at (59.0, 3.50)
- added R310: 0R5, Resistor_THT:R_Axial_DIN0411_L9.9mm_D3.6mm_P5.08mm_Vertical, F.Cu at (57.5, 33.0)
- added R401: R, Resistor_THT:R_Axial_DIN0204_L3.6mm_D1.6mm_P2.54mm_Vertical, F.Cu at (66.5, 70.0)
- added R402: R, Resistor_THT:R_Axial_DIN0204_L3.6mm_D1.6mm_P2.54mm_Vertical, F.Cu at (69.5, 67.5)
- added R403: 1, Resistor_THT:R_Axial_DIN0204_L3.6mm_D1.6mm_P2.54mm_Vertical, F.Cu at (72.5, 70.0)
- added R404: R, Resistor_THT:R_Axial_DIN0204_L3.6mm_D1.6mm_P2.54mm_Vertical, F.Cu at (66.5, 62.0)
- added R405: R, Resistor_THT:R_Axial_DIN0204_L3.6mm_D1.6mm_P2.54mm_Vertical, F.Cu at (69.5, 64.5)
- added R406: 1, Resistor_THT:R_Axial_DIN0204_L3.6mm_D1.6mm_P2.54mm_Vertical, F.Cu at (72.5, 62.0)
- added R407: 0R5, Resistor_THT:R_Axial_DIN0411_L9.9mm_D3.6mm_P5.08mm_Vertical, F.Cu at (27.4, 57.7)
- added R408: 0R5, Resistor_THT:R_Axial_DIN0411_L9.9mm_D3.6mm_P5.08mm_Vertical, F.Cu at (27.4, 52.6)
- added R409: 0R5, Resistor_THT:R_Axial_DIN0411_L9.9mm_D3.6mm_P5.08mm_Vertical, F.Cu at (59.0, 39.5)
- added R410: 0R5, Resistor_THT:R_Axial_DIN0411_L9.9mm_D3.6mm_P5.08mm_Vertical, F.Cu at (57.5, 69.0)
- added R601: R, Resistor_THT:R_Axial_DIN0204_L3.6mm_D1.6mm_P2.54mm_Vertical, F.Cu at (66.5, 106.0)
- added R602: R, Resistor_THT:R_Axial_DIN0204_L3.6mm_D1.6mm_P2.54mm_Vertical, F.Cu at (69.5, 103.5)
- added R603: 1, Resistor_THT:R_Axial_DIN0204_L3.6mm_D1.6mm_P2.54mm_Vertical, F.Cu at (72.5, 106.0)
- added R604: R, Resistor_THT:R_Axial_DIN0204_L3.6mm_D1.6mm_P2.54mm_Vertical, F.Cu at (66.5, 98.0)
- added R605: R, Resistor_THT:R_Axial_DIN0204_L3.6mm_D1.6mm_P2.54mm_Vertical, F.Cu at (69.5, 100.5)
- added R606: 1, Resistor_THT:R_Axial_DIN0204_L3.6mm_D1.6mm_P2.54mm_Vertical, F.Cu at (72.5, 98.0)
- added R607: 0R5, Resistor_THT:R_Axial_DIN0411_L9.9mm_D3.6mm_P5.08mm_Vertical, F.Cu at (27.4, 93.7)
- added R608: 0R5, Resistor_THT:R_Axial_DIN0411_L9.9mm_D3.6mm_P5.08mm_Vertical, F.Cu at (27.4, 88.6)
- added R609: 0R5, Resistor_THT:R_Axial_DIN0411_L9.9mm_D3.6mm_P5.08mm_Vertical, F.Cu at (59.0, 75.5)
- added R610: 0R5, Resistor_THT:R_Axial_DIN0411_L9.9mm_D3.6mm_P5.08mm_Vertical, F.Cu at (57.5, 105.0)
- added R701: R, Resistor_THT:R_Axial_DIN0204_L3.6mm_D1.6mm_P2.54mm_Vertical, F.Cu at (66.5, 142.0)
- added R702: R, Resistor_THT:R_Axial_DIN0204_L3.6mm_D1.6mm_P2.54mm_Vertical, F.Cu at (69.5, 139.5)
- added R703: 1, Resistor_THT:R_Axial_DIN0204_L3.6mm_D1.6mm_P2.54mm_Vertical, F.Cu at (72.5, 142.0)
- added R704: R, Resistor_THT:R_Axial_DIN0204_L3.6mm_D1.6mm_P2.54mm_Vertical, F.Cu at (66.5, 134.0)
- added R705: R, Resistor_THT:R_Axial_DIN0204_L3.6mm_D1.6mm_P2.54mm_Vertical, F.Cu at (69.5, 136.5)
- added R706: 1, Resistor_THT:R_Axial_DIN0204_L3.6mm_D1.6mm_P2.54mm_Vertical, F.Cu at (72.5, 134.0)
- added R707: 0R5, Resistor_THT:R_Axial_DIN0411_L9.9mm_D3.6mm_P5.08mm_Vertical, F.Cu at (27.4, 129.7)
- added R708: 0R5, Resistor_THT:R_Axial_DIN0411_L9.9mm_D3.6mm_P5.08mm_Vertical, F.Cu at (27.4, 124.6)
- added R709: 0R5, Resistor_THT:R_Axial_DIN0411_L9.9mm_D3.6mm_P5.08mm_Vertical, F.Cu at (59.0, 111.5)
- added R710: 0R5, Resistor_THT:R_Axial_DIN0411_L9.9mm_D3.6mm_P5.08mm_Vertical, F.Cu at (57.5, 141.0)
- added R801: R, Resistor_THT:R_Axial_DIN0204_L3.6mm_D1.6mm_P2.54mm_Vertical, F.Cu at (66.5, 178.0)
- added R802: R, Resistor_THT:R_Axial_DIN0204_L3.6mm_D1.6mm_P2.54mm_Vertical, F.Cu at (69.5, 175.5)
- added R803: 1, Resistor_THT:R_Axial_DIN0204_L3.6mm_D1.6mm_P2.54mm_Vertical, F.Cu at (72.5, 178.0)
- added R804: R, Resistor_THT:R_Axial_DIN0204_L3.6mm_D1.6mm_P2.54mm_Vertical, F.Cu at (66.5, 170.0)
- added R805: R, Resistor_THT:R_Axial_DIN0204_L3.6mm_D1.6mm_P2.54mm_Vertical, F.Cu at (69.5, 172.5)
- added R806: 1, Resistor_THT:R_Axial_DIN0204_L3.6mm_D1.6mm_P2.54mm_Vertical, F.Cu at (72.5, 170.0)
- added R807: 0R5, Resistor_THT:R_Axial_DIN0411_L9.9mm_D3.6mm_P5.08mm_Vertical, F.Cu at (27.4, 165.7)
- added R808: 0R5, Resistor_THT:R_Axial_DIN0411_L9.9mm_D3.6mm_P5.08mm_Vertical, F.Cu at (27.4, 160.6)
- added R809: 0R5, Resistor_THT:R_Axial_DIN0411_L9.9mm_D3.6mm_P5.08mm_Vertical, F.Cu at (59.0, 147.5)
- added R810: 0R5, Resistor_THT:R_Axial_DIN0411_L9.9mm_D3.6mm_P5.08mm_Vertical, F.Cu at (57.5, 177.0)
- added R901: R, Resistor_THT:R_Axial_DIN0204_L3.6mm_D1.6mm_P2.54mm_Vertical, F.Cu at (66.5, 214.0)
- added R902: R, Resistor_THT:R_Axial_DIN0204_L3.6mm_D1.6mm_P2.54mm_Vertical, F.Cu at (69.5, 211.5)
- added R903: 1, Resistor_THT:R_Axial_DIN0204_L3.6mm_D1.6mm_P2.54mm_Vertical, F.Cu at (72.5, 214.0)
- added R904: R, Resistor_THT:R_Axial_DIN0204_L3.6mm_D1.6mm_P2.54mm_Vertical, F.Cu at (66.5, 206.0)
- added R905: R, Resistor_THT:R_Axial_DIN0204_L3.6mm_D1.6mm_P2.54mm_Vertical, F.Cu at (69.5, 208.5)
- added R906: 1, Resistor_THT:R_Axial_DIN0204_L3.6mm_D1.6mm_P2.54mm_Vertical, F.Cu at (72.5, 206.0)
- added R907: 0R5, Resistor_THT:R_Axial_DIN0411_L9.9mm_D3.6mm_P5.08mm_Vertical, F.Cu at (27.4, 201.7)
- added R908: 0R5, Resistor_THT:R_Axial_DIN0411_L9.9mm_D3.6mm_P5.08mm_Vertical, F.Cu at (27.4, 196.6)
- added R909: 0R5, Resistor_THT:R_Axial_DIN0411_L9.9mm_D3.6mm_P5.08mm_Vertical, F.Cu at (59.0, 183.5)
- added R910: 0R5, Resistor_THT:R_Axial_DIN0411_L9.9mm_D3.6mm_P5.08mm_Vertical, F.Cu at (57.5, 213.0)
- added U301: DRV8823, Package_SO:TSSOP-48_6.1x12.5mm_P0.5mm, F.Cu at (51.6, 17.2)
- added U401: DRV8823, Package_SO:TSSOP-48_6.1x12.5mm_P0.5mm, F.Cu at (51.6, 53.2)
- added U601: DRV8823, Package_SO:TSSOP-48_6.1x12.5mm_P0.5mm, F.Cu at (51.6, 89.2)
- added U701: DRV8823, Package_SO:TSSOP-48_6.1x12.5mm_P0.5mm, F.Cu at (51.6, 125.2)
- added U801: DRV8823, Package_SO:TSSOP-48_6.1x12.5mm_P0.5mm, F.Cu at (51.6, 161.2)
- added U901: DRV8823, Package_SO:TSSOP-48_6.1x12.5mm_P0.5mm, F.Cu at (51.6, 197.2)
- C1002, C1102, C1202, C1302, C1402, C1502, C1602, C1702: value 100nF 6,3V -> 100nF; footprint Capacitor_SMD:C_0201_0603Metric -> Capacitor_THT:C_Disc_D8.0mm_W5.0mm_P5.00mm
- C1003, C1103, C1203, C1303, C1403, C1503, C1603, C1703: value 100nF -> 100nF 6,3V; footprint Capacitor_THT:C_Disc_D8.0mm_W5.0mm_P5.00mm -> Capacitor_SMD:C_0201_0603Metric
- C1004, C1006, C1104, C1106, C1204, C1206, C1304, C1306, C1404, C1406, C1504, C1506, C1604, C1606, C1704, C1706: moved to F.Cu
- J1001, J1101, J1201, J1301, J1401, J1501, J1601, J1701: value Screw_Terminal_01x04 -> Screw_Terminal_01x08; footprint Connector_Phoenix_MC_HighVoltage:PhoenixContact_MCV_1,5_4-G-5.08_1x04_P5.08mm_Vertical -> TerminalBlock_Phoenix:TerminalBlock_Phoenix_PT-1,5-8-3.5-H_1x08_P3.50mm_Horizontal
- J1002, J1102, J1202, J1302, J1402, J1502, J1602, J1702: value Screw_Terminal_01x04 -> Conn_01x10_Male; footprint Connector_Phoenix_MC_HighVoltage:PhoenixContact_MCV_1,5_4-G-5.08_1x04_P5.08mm_Vertical -> Connector_PinHeader_1.00mm:PinHeader_1x10_P1.00mm_Vertical
- R1001, R1002, R1004, R1101, R1102, R1104, R1201, R1202, R1204, R1301, R1302, R1304, R1401, R1402, R1404, R1501, R1502, R1504, R1601, R1602, R1604, R1701, R1702, R1704: value 0R5 -> R; footprint Resistor_THT:R_Axial_DIN0411_L9.9mm_D3.6mm_P5.08mm_Vertical -> Resistor_THT:R_Axial_DIN0204_L3.6mm_D1.6mm_P2.54mm_Vertical
- R1003, R1103, R1203, R1303, R1403, R1503, R1603, R1703: value 0R5 -> 1; footprint Resistor_THT:R_Axial_DIN0411_L9.9mm_D3.6mm_P5.08mm_Vertical -> Resistor_THT:R_Axial_DIN0204_L3.6mm_D1.6mm_P2.54mm_Vertical
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Connections:
- C1001 pad 1: +28V -> Net-(C1001-Pad1)
- C1002 pad 1: Net-(C1002-Pad1) -> Net-(C1001-Pad1)
- C1003 pad 1: +28V -> Net-(C1003-Pad1)
- C1004 pad 1: /Steuer5 -> Net-(C1004-Pad1)
- C1005 pad 1: +28V -> Net-(C1001-Pad1)
- C1006 pad 1: /Steuer6 -> Net-(C1006-Pad1)
- C1008 pad 2: +28V -> Net-(C1001-Pad1)
- C1101 pad 1: +28V -> Net-(C1101-Pad1)
- C1102 pad 1: Net-(C1102-Pad1) -> Net-(C1101-Pad1)
- C1103 pad 1: +28V -> Net-(C1103-Pad1)
- C1104 pad 1: /Steuer5 -> Net-(C1104-Pad1)
- C1105 pad 1: +28V -> Net-(C1101-Pad1)
- C1106 pad 1: /Steuer6 -> Net-(C1106-Pad1)
- C1108 pad 2: +28V -> Net-(C1101-Pad1)
- C1201 pad 1: +28V -> Net-(C1201-Pad1)
- C1202 pad 1: Net-(C1202-Pad1) -> Net-(C1201-Pad1)
- C1203 pad 1: +28V -> Net-(C1203-Pad1)
- C1204 pad 1: /Steuer5 -> Net-(C1204-Pad1)
- C1205 pad 1: +28V -> Net-(C1201-Pad1)
- C1206 pad 1: /Steuer6 -> Net-(C1206-Pad1)
- C1208 pad 2: +28V -> Net-(C1201-Pad1)
- C1301 pad 1: +28V -> Net-(C1301-Pad1)
- C1302 pad 1: Net-(C1302-Pad1) -> Net-(C1301-Pad1)
- C1303 pad 1: +28V -> Net-(C1303-Pad1)
- C1304 pad 1: /Steuer5 -> Net-(C1304-Pad1)
- C1305 pad 1: +28V -> Net-(C1301-Pad1)
- C1306 pad 1: /Steuer6 -> Net-(C1306-Pad1)
- C1308 pad 2: +28V -> Net-(C1301-Pad1)
- C1401 pad 1: +28V -> Net-(C1401-Pad1)
- C1402 pad 1: Net-(C1402-Pad1) -> Net-(C1401-Pad1)
- C1403 pad 1: +28V -> Net-(C1403-Pad1)
- C1404 pad 1: /Steuer5 -> Net-(C1404-Pad1)
- C1405 pad 1: +28V -> Net-(C1401-Pad1)
- C1406 pad 1: /Steuer6 -> Net-(C1406-Pad1)
- C1408 pad 2: +28V -> Net-(C1401-Pad1)
- C1501 pad 1: +28V -> Net-(C1501-Pad1)
- C1502 pad 1: Net-(C1502-Pad1) -> Net-(C1501-Pad1)
- C1503 pad 1: +28V -> Net-(C1503-Pad1)
- C1504 pad 1: /Steuer5 -> Net-(C1504-Pad1)
- C1505 pad 1: +28V -> Net-(C1501-Pad1)
- C1506 pad 1: /Steuer6 -> Net-(C1506-Pad1)
- C1508 pad 2: +28V -> Net-(C1501-Pad1)
- C1601 pad 1: +28V -> Net-(C1601-Pad1)
- C1602 pad 1: Net-(C1602-Pad1) -> Net-(C1601-Pad1)
- C1603 pad 1: +28V -> Net-(C1603-Pad1)
- C1604 pad 1: /Steuer5 -> Net-(C1604-Pad1)
- C1605 pad 1: +28V -> Net-(C1601-Pad1)
- C1606 pad 1: /Steuer6 -> Net-(C1606-Pad1)
- C1608 pad 2: +28V -> Net-(C1601-Pad1)
- C1701 pad 1: +28V -> Net-(C1701-Pad1)
- C1702 pad 1: Net-(C1702-Pad1) -> Net-(C1701-Pad1)
- C1703 pad 1: +28V -> Net-(C1703-Pad1)
- C1704 pad 1: /Steuer5 -> Net-(C1704-Pad1)
- C1705 pad 1: +28V -> Net-(C1701-Pad1)
- C1706 pad 1: /Steuer6 -> Net-(C1706-Pad1)
- C1708 pad 2: +28V -> Net-(C1701-Pad1)
- J1001 pad 1: /Motortreiber0/MA1 -> /Motortreiber14/MC1
- J1001 pad 2: /Motortreiber0/MA2 -> /Motortreiber14/MC2
- J1001 pad 3: /Motortreiber0/MB2 -> /Motortreiber14/MD1
- J1001 pad 4: /Motortreiber0/MB1 -> /Motortreiber14/MD2
- J1002 pad 1: /Motortreiber0/MC1 -> /Steuer1
- J1002 pad 2: /Motortreiber0/MC2 -> /Steuer0
- J1002 pad 3: /Motortreiber0/MD1 -> /Steuer4
- J1002 pad 4: /Motortreiber0/MD2 -> GND
- J1101 pad 1: /Motortreiber1/MA1 -> /Motortreiber13/MC1
- J1101 pad 2: /Motortreiber1/MA2 -> /Motortreiber13/MC2
- J1101 pad 3: /Motortreiber1/MB2 -> /Motortreiber13/MD1
- J1101 pad 4: /Motortreiber1/MB1 -> /Motortreiber13/MD2
- J1102 pad 1: /Motortreiber1/MC1 -> /Steuer1
- J1102 pad 2: /Motortreiber1/MC2 -> /Steuer0
- J1102 pad 3: /Motortreiber1/MD1 -> /Steuer4
- J1102 pad 4: /Motortreiber1/MD2 -> GND
- J1201 pad 1: /Motortreiber2/MA1 -> /Motortreiber12/MC1
- J1201 pad 2: /Motortreiber2/MA2 -> /Motortreiber12/MC2
- J1201 pad 3: /Motortreiber2/MB2 -> /Motortreiber12/MD1
- J1201 pad 4: /Motortreiber2/MB1 -> /Motortreiber12/MD2
- J1202 pad 1: /Motortreiber2/MC1 -> /Steuer1
- J1202 pad 2: /Motortreiber2/MC2 -> /Steuer0
- J1202 pad 3: /Motortreiber2/MD1 -> /Steuer4
- J1202 pad 4: /Motortreiber2/MD2 -> GND
- J1301 pad 1: /Motortreiber3/MA1 -> /Motortreiber2/MC1
- J1301 pad 2: /Motortreiber3/MA2 -> /Motortreiber2/MC2
- J1301 pad 3: /Motortreiber3/MB2 -> /Motortreiber2/MD1
- J1301 pad 4: /Motortreiber3/MB1 -> /Motortreiber2/MD2
- J1302 pad 1: /Motortreiber3/MC1 -> /Steuer1
- J1302 pad 2: /Motortreiber3/MC2 -> /Steuer0
- J1302 pad 3: /Motortreiber3/MD1 -> /Steuer4
- J1302 pad 4: /Motortreiber3/MD2 -> GND
- J1401 pad 1: /Motortreiber4/MA1 -> /Motortreiber7/MC1
- J1401 pad 2: /Motortreiber4/MA2 -> /Motortreiber7/MC2
- J1401 pad 3: /Motortreiber4/MB2 -> /Motortreiber7/MD1
- J1401 pad 4: /Motortreiber4/MB1 -> /Motortreiber7/MD2
- J1402 pad 1: /Motortreiber4/MC1 -> /Steuer1
- J1402 pad 2: /Motortreiber4/MC2 -> /Steuer0
- J1402 pad 3: /Motortreiber4/MD1 -> /Steuer4
- J1402 pad 4: /Motortreiber4/MD2 -> GND
- J1501 pad 1: /Motortreiber5/MA1 -> /Motortreiber8/MC1
- J1501 pad 2: /Motortreiber5/MA2 -> /Motortreiber8/MC2
- J1501 pad 3: /Motortreiber5/MB2 -> /Motortreiber8/MD1
- J1501 pad 4: /Motortreiber5/MB1 -> /Motortreiber8/MD2
- J1502 pad 1: /Motortreiber5/MC1 -> /Steuer1
- J1502 pad 2: /Motortreiber5/MC2 -> /Steuer0
- J1502 pad 3: /Motortreiber5/MD1 -> /Steuer4
- J1502 pad 4: /Motortreiber5/MD2 -> GND
- J1601 pad 1: /Motortreiber6/MA1 -> /Motortreiber4/MC1
- J1601 pad 2: /Motortreiber6/MA2 -> /Motortreiber4/MC2
- J1601 pad 3: /Motortreiber6/MB2 -> /Motortreiber4/MD1
- J1601 pad 4: /Motortreiber6/MB1 -> /Motortreiber4/MD2
- J1602 pad 1: /Motortreiber6/MC1 -> /Steuer1
- J1602 pad 2: /Motortreiber6/MC2 -> /Steuer0
- J1602 pad 3: /Motortreiber6/MD1 -> /Steuer4
- J1602 pad 4: /Motortreiber6/MD2 -> GND
- J1701 pad 1: /Motortreiber7/MA1 -> /Motortreiber10/MC1
- J1701 pad 2: /Motortreiber7/MA2 -> /Motortreiber10/MC2
- J1701 pad 3: /Motortreiber7/MB2 -> /Motortreiber10/MD1
- J1701 pad 4: /Motortreiber7/MB1 -> /Motortreiber10/MD2
- J1702 pad 1: /Motortreiber7/MC1 -> /Steuer1
- J1702 pad 2: /Motortreiber7/MC2 -> /Steuer0
- J1702 pad 3: /Motortreiber7/MD1 -> /Steuer4
- J1702 pad 4: /Motortreiber7/MD2 -> GND
- R1001 pad 1: /Motortreiber0/MDR -> Net-(C1003-Pad1)
- R1001 pad 2: GND -> Net-(C1006-Pad1)
- R1002 pad 1: /Motortreiber0/MAR -> Net-(C1006-Pad1)
- R1003 pad 1: GND -> /Steuer6
- R1003 pad 2: /Motortreiber0/MBR -> Net-(C1006-Pad1)
- R1004 pad 1: GND -> Net-(C1003-Pad1)
- R1004 pad 2: /Motortreiber0/MCR -> Net-(C1004-Pad1)
- R1101 pad 1: /Motortreiber1/MDR -> Net-(C1103-Pad1)
- R1101 pad 2: GND -> Net-(C1106-Pad1)
- R1102 pad 1: /Motortreiber1/MAR -> Net-(C1106-Pad1)
- R1103 pad 1: GND -> /Steuer6
- R1103 pad 2: /Motortreiber1/MBR -> Net-(C1106-Pad1)
- R1104 pad 1: GND -> Net-(C1103-Pad1)
- R1104 pad 2: /Motortreiber1/MCR -> Net-(C1104-Pad1)
- R1201 pad 1: /Motortreiber2/MDR -> Net-(C1203-Pad1)
- R1201 pad 2: GND -> Net-(C1206-Pad1)
- R1202 pad 1: /Motortreiber2/MAR -> Net-(C1206-Pad1)
- R1203 pad 1: GND -> /Steuer6
- R1203 pad 2: /Motortreiber2/MBR -> Net-(C1206-Pad1)
- R1204 pad 1: GND -> Net-(C1203-Pad1)
- R1204 pad 2: /Motortreiber2/MCR -> Net-(C1204-Pad1)
- R1301 pad 1: /Motortreiber3/MDR -> Net-(C1303-Pad1)
- R1301 pad 2: GND -> Net-(C1306-Pad1)
- R1302 pad 1: /Motortreiber3/MAR -> Net-(C1306-Pad1)
- R1303 pad 1: GND -> /Steuer6
- R1303 pad 2: /Motortreiber3/MBR -> Net-(C1306-Pad1)
- R1304 pad 1: GND -> Net-(C1303-Pad1)
- R1304 pad 2: /Motortreiber3/MCR -> Net-(C1304-Pad1)
- R1401 pad 1: /Motortreiber4/MDR -> Net-(C1403-Pad1)
- R1401 pad 2: GND -> Net-(C1406-Pad1)
- R1402 pad 1: /Motortreiber4/MAR -> Net-(C1406-Pad1)
- R1403 pad 1: GND -> /Steuer6
- R1403 pad 2: /Motortreiber4/MBR -> Net-(C1406-Pad1)
- R1404 pad 1: GND -> Net-(C1403-Pad1)
- R1404 pad 2: /Motortreiber4/MCR -> Net-(C1404-Pad1)
- R1501 pad 1: /Motortreiber5/MDR -> Net-(C1503-Pad1)
- R1501 pad 2: GND -> Net-(C1506-Pad1)
- R1502 pad 1: /Motortreiber5/MAR -> Net-(C1506-Pad1)
- R1503 pad 1: GND -> /Steuer6
- R1503 pad 2: /Motortreiber5/MBR -> Net-(C1506-Pad1)
- R1504 pad 1: GND -> Net-(C1503-Pad1)
- R1504 pad 2: /Motortreiber5/MCR -> Net-(C1504-Pad1)
- R1601 pad 1: /Motortreiber6/MDR -> Net-(C1603-Pad1)
- R1601 pad 2: GND -> Net-(C1606-Pad1)
- R1602 pad 1: /Motortreiber6/MAR -> Net-(C1606-Pad1)
- R1603 pad 1: GND -> /Steuer6
- R1603 pad 2: /Motortreiber6/MBR -> Net-(C1606-Pad1)
- R1604 pad 1: GND -> Net-(C1603-Pad1)
- R1604 pad 2: /Motortreiber6/MCR -> Net-(C1604-Pad1)
- R1701 pad 1: /Motortreiber7/MDR -> Net-(C1703-Pad1)
- R1701 pad 2: GND -> Net-(C1706-Pad1)
- R1702 pad 1: /Motortreiber7/MAR -> Net-(C1706-Pad1)
- R1703 pad 1: GND -> /Steuer6
- R1703 pad 2: /Motortreiber7/MBR -> Net-(C1706-Pad1)
- R1704 pad 1: GND -> Net-(C1703-Pad1)
- R1704 pad 2: /Motortreiber7/MCR -> Net-(C1704-Pad1)
- U1001 pad 1: +28V -> Net-(C1001-Pad1)
- U1001 pad 16: Net-(C1002-Pad1) -> Net-(C1003-Pad1)
- U1001 pad 17: /Steuer5 -> Net-(C1004-Pad1)
- U1001 pad 18: /Steuer6 -> Net-(C1006-Pad1)
- U1001 pad 19: Net-(U1001-Pad19) -> (no net)
- U1001 pad 2: +28V -> Net-(C1001-Pad1)
- U1001 pad 20: /Motortreiber0/MD2 -> /Motortreiber14/MD2
- U1001 pad 21: /Motortreiber0/MDR -> /Motortreiber14/MDR
- U1001 pad 22: /Motortreiber0/MD1 -> /Motortreiber14/MD1
- U1001 pad 23: +28V -> Net-(C1001-Pad1)
- U1001 pad 24: +28V -> Net-(C1001-Pad1)
- U1001 pad 25: /Motortreiber0/MC2 -> /Motortreiber14/MC2
- U1001 pad 26: /Motortreiber0/MCR -> /Motortreiber14/MCR
- U1001 pad 27: /Motortreiber0/MC1 -> /Motortreiber14/MC1
- U1001 pad 28: Net-(U1001-Pad28) -> (no net)
- U1001 pad 29: Net-(U1001-Pad29) -> (no net)
- U1001 pad 3: /Motortreiber0/MA2 -> /Motortreiber14/MA2
- U1001 pad 30: /Strobe0 -> /Strobe14
- U1001 pad 32: Net-(U1001-Pad32) -> (no net)
- U1001 pad 4: /Motortreiber0/MAR -> /Motortreiber14/MAR
- U1001 pad 40: Net-(U1001-Pad40) -> (no net)
- U1001 pad 41: Net-(U1001-Pad41) -> (no net)
- U1001 pad 44: Net-(U1001-Pad44) -> (no net)
- U1001 pad 46: /Motortreiber0/MB1 -> /Motortreiber14/MB1
- U1001 pad 47: /Motortreiber0/MBR -> /Motortreiber14/MBR
- U1001 pad 48: /Motortreiber0/MB2 -> /Motortreiber14/MB2
- U1001 pad 5: /Motortreiber0/MA1 -> /Motortreiber14/MA1
- U1001 pad 6: Net-(U1001-Pad6) -> (no net)
- U1101 pad 1: +28V -> Net-(C1101-Pad1)
- U1101 pad 16: Net-(C1102-Pad1) -> Net-(C1103-Pad1)
- U1101 pad 17: /Steuer5 -> Net-(C1104-Pad1)
- U1101 pad 18: /Steuer6 -> Net-(C1106-Pad1)
- U1101 pad 19: Net-(U1101-Pad19) -> (no net)
- U1101 pad 2: +28V -> Net-(C1101-Pad1)
- U1101 pad 20: /Motortreiber1/MD2 -> /Motortreiber13/MD2
- U1101 pad 21: /Motortreiber1/MDR -> /Motortreiber13/MDR
- U1101 pad 22: /Motortreiber1/MD1 -> /Motortreiber13/MD1
- U1101 pad 23: +28V -> Net-(C1101-Pad1)
- U1101 pad 24: +28V -> Net-(C1101-Pad1)
- U1101 pad 25: /Motortreiber1/MC2 -> /Motortreiber13/MC2
- U1101 pad 26: /Motortreiber1/MCR -> /Motortreiber13/MCR
- U1101 pad 27: /Motortreiber1/MC1 -> /Motortreiber13/MC1
- U1101 pad 28: Net-(U1101-Pad28) -> (no net)
- U1101 pad 29: Net-(U1101-Pad29) -> (no net)
- U1101 pad 3: /Motortreiber1/MA2 -> /Motortreiber13/MA2
- U1101 pad 30: /Strobe1 -> /Strobe13
- U1101 pad 32: Net-(U1101-Pad32) -> (no net)
- U1101 pad 4: /Motortreiber1/MAR -> /Motortreiber13/MAR
- U1101 pad 40: Net-(U1101-Pad40) -> (no net)
- U1101 pad 41: Net-(U1101-Pad41) -> (no net)
- U1101 pad 44: Net-(U1101-Pad44) -> (no net)
- U1101 pad 46: /Motortreiber1/MB1 -> /Motortreiber13/MB1
- U1101 pad 47: /Motortreiber1/MBR -> /Motortreiber13/MBR
- U1101 pad 48: /Motortreiber1/MB2 -> /Motortreiber13/MB2
- U1101 pad 5: /Motortreiber1/MA1 -> /Motortreiber13/MA1
- U1101 pad 6: Net-(U1101-Pad6) -> (no net)
- U1201 pad 1: +28V -> Net-(C1201-Pad1)
- U1201 pad 16: Net-(C1202-Pad1) -> Net-(C1203-Pad1)
- U1201 pad 17: /Steuer5 -> Net-(C1204-Pad1)
- U1201 pad 18: /Steuer6 -> Net-(C1206-Pad1)
- U1201 pad 19: Net-(U1201-Pad19) -> (no net)
- U1201 pad 2: +28V -> Net-(C1201-Pad1)
- U1201 pad 20: /Motortreiber2/MD2 -> /Motortreiber12/MD2
- U1201 pad 21: /Motortreiber2/MDR -> /Motortreiber12/MDR
- U1201 pad 22: /Motortreiber2/MD1 -> /Motortreiber12/MD1
- U1201 pad 23: +28V -> Net-(C1201-Pad1)
- U1201 pad 24: +28V -> Net-(C1201-Pad1)
- U1201 pad 25: /Motortreiber2/MC2 -> /Motortreiber12/MC2
- U1201 pad 26: /Motortreiber2/MCR -> /Motortreiber12/MCR
- U1201 pad 27: /Motortreiber2/MC1 -> /Motortreiber12/MC1
- U1201 pad 28: Net-(U1201-Pad28) -> (no net)
- U1201 pad 29: Net-(U1201-Pad29) -> (no net)
- U1201 pad 3: /Motortreiber2/MA2 -> /Motortreiber12/MA2
- U1201 pad 30: /Strobe2 -> /Strobe12
- U1201 pad 32: Net-(U1201-Pad32) -> (no net)
- U1201 pad 4: /Motortreiber2/MAR -> /Motortreiber12/MAR
- U1201 pad 40: Net-(U1201-Pad40) -> (no net)
- U1201 pad 41: Net-(U1201-Pad41) -> (no net)
- U1201 pad 44: Net-(U1201-Pad44) -> (no net)
- U1201 pad 46: /Motortreiber2/MB1 -> /Motortreiber12/MB1
- U1201 pad 47: /Motortreiber2/MBR -> /Motortreiber12/MBR
- U1201 pad 48: /Motortreiber2/MB2 -> /Motortreiber12/MB2
- U1201 pad 5: /Motortreiber2/MA1 -> /Motortreiber12/MA1
- U1201 pad 6: Net-(U1201-Pad6) -> (no net)
- U1301 pad 1: +28V -> Net-(C1301-Pad1)
- U1301 pad 16: Net-(C1302-Pad1) -> Net-(C1303-Pad1)
- U1301 pad 17: /Steuer5 -> Net-(C1304-Pad1)
- U1301 pad 18: /Steuer6 -> Net-(C1306-Pad1)
- U1301 pad 19: Net-(U1301-Pad19) -> (no net)
- U1301 pad 2: +28V -> Net-(C1301-Pad1)
- U1301 pad 20: /Motortreiber3/MD2 -> /Motortreiber2/MD2
- U1301 pad 21: /Motortreiber3/MDR -> /Motortreiber2/MDR
- U1301 pad 22: /Motortreiber3/MD1 -> /Motortreiber2/MD1
- U1301 pad 23: +28V -> Net-(C1301-Pad1)
- U1301 pad 24: +28V -> Net-(C1301-Pad1)
- U1301 pad 25: /Motortreiber3/MC2 -> /Motortreiber2/MC2
- U1301 pad 26: /Motortreiber3/MCR -> /Motortreiber2/MCR
- U1301 pad 27: /Motortreiber3/MC1 -> /Motortreiber2/MC1
- U1301 pad 28: Net-(U1301-Pad28) -> (no net)
- U1301 pad 29: Net-(U1301-Pad29) -> (no net)
- U1301 pad 3: /Motortreiber3/MA2 -> /Motortreiber2/MA2
- U1301 pad 30: /Strobe3 -> /Strobe2
- U1301 pad 32: Net-(U1301-Pad32) -> (no net)
- U1301 pad 4: /Motortreiber3/MAR -> /Motortreiber2/MAR
- U1301 pad 40: Net-(U1301-Pad40) -> (no net)
- U1301 pad 41: Net-(U1301-Pad41) -> (no net)
- U1301 pad 44: Net-(U1301-Pad44) -> (no net)
- U1301 pad 46: /Motortreiber3/MB1 -> /Motortreiber2/MB1
- U1301 pad 47: /Motortreiber3/MBR -> /Motortreiber2/MBR
- U1301 pad 48: /Motortreiber3/MB2 -> /Motortreiber2/MB2
- U1301 pad 5: /Motortreiber3/MA1 -> /Motortreiber2/MA1
- U1301 pad 6: Net-(U1301-Pad6) -> (no net)
- U1401 pad 1: +28V -> Net-(C1401-Pad1)
- U1401 pad 16: Net-(C1402-Pad1) -> Net-(C1403-Pad1)
- U1401 pad 17: /Steuer5 -> Net-(C1404-Pad1)
- U1401 pad 18: /Steuer6 -> Net-(C1406-Pad1)
- U1401 pad 19: Net-(U1401-Pad19) -> (no net)
- U1401 pad 2: +28V -> Net-(C1401-Pad1)
- U1401 pad 20: /Motortreiber4/MD2 -> /Motortreiber7/MD2
- U1401 pad 21: /Motortreiber4/MDR -> /Motortreiber7/MDR
- U1401 pad 22: /Motortreiber4/MD1 -> /Motortreiber7/MD1
- U1401 pad 23: +28V -> Net-(C1401-Pad1)
- U1401 pad 24: +28V -> Net-(C1401-Pad1)
- U1401 pad 25: /Motortreiber4/MC2 -> /Motortreiber7/MC2
- U1401 pad 26: /Motortreiber4/MCR -> /Motortreiber7/MCR
- U1401 pad 27: /Motortreiber4/MC1 -> /Motortreiber7/MC1
- U1401 pad 28: Net-(U1401-Pad28) -> (no net)
- U1401 pad 29: Net-(U1401-Pad29) -> (no net)
- U1401 pad 3: /Motortreiber4/MA2 -> /Motortreiber7/MA2
- U1401 pad 30: /Strobe4 -> /Strobe7
- U1401 pad 32: Net-(U1401-Pad32) -> (no net)
- U1401 pad 4: /Motortreiber4/MAR -> /Motortreiber7/MAR
- U1401 pad 40: Net-(U1401-Pad40) -> (no net)
- U1401 pad 41: Net-(U1401-Pad41) -> (no net)
- U1401 pad 44: Net-(U1401-Pad44) -> (no net)
- U1401 pad 46: /Motortreiber4/MB1 -> /Motortreiber7/MB1
- U1401 pad 47: /Motortreiber4/MBR -> /Motortreiber7/MBR
- U1401 pad 48: /Motortreiber4/MB2 -> /Motortreiber7/MB2
- U1401 pad 5: /Motortreiber4/MA1 -> /Motortreiber7/MA1
- U1401 pad 6: Net-(U1401-Pad6) -> (no net)
- U1501 pad 1: +28V -> Net-(C1501-Pad1)
- U1501 pad 16: Net-(C1502-Pad1) -> Net-(C1503-Pad1)
- U1501 pad 17: /Steuer5 -> Net-(C1504-Pad1)
- U1501 pad 18: /Steuer6 -> Net-(C1506-Pad1)
- U1501 pad 19: Net-(U1501-Pad19) -> (no net)
- U1501 pad 2: +28V -> Net-(C1501-Pad1)
- U1501 pad 20: /Motortreiber5/MD2 -> /Motortreiber8/MD2
- U1501 pad 21: /Motortreiber5/MDR -> /Motortreiber8/MDR
- U1501 pad 22: /Motortreiber5/MD1 -> /Motortreiber8/MD1
- U1501 pad 23: +28V -> Net-(C1501-Pad1)
- U1501 pad 24: +28V -> Net-(C1501-Pad1)
- U1501 pad 25: /Motortreiber5/MC2 -> /Motortreiber8/MC2
- U1501 pad 26: /Motortreiber5/MCR -> /Motortreiber8/MCR
- U1501 pad 27: /Motortreiber5/MC1 -> /Motortreiber8/MC1
- U1501 pad 28: Net-(U1501-Pad28) -> (no net)
- U1501 pad 29: Net-(U1501-Pad29) -> (no net)
- U1501 pad 3: /Motortreiber5/MA2 -> /Motortreiber8/MA2
- U1501 pad 30: /Strobe5 -> /Strobe8
- U1501 pad 32: Net-(U1501-Pad32) -> (no net)
- U1501 pad 4: /Motortreiber5/MAR -> /Motortreiber8/MAR
- U1501 pad 40: Net-(U1501-Pad40) -> (no net)
- U1501 pad 41: Net-(U1501-Pad41) -> (no net)
- U1501 pad 44: Net-(U1501-Pad44) -> (no net)
- U1501 pad 46: /Motortreiber5/MB1 -> /Motortreiber8/MB1
- U1501 pad 47: /Motortreiber5/MBR -> /Motortreiber8/MBR
- U1501 pad 48: /Motortreiber5/MB2 -> /Motortreiber8/MB2
- U1501 pad 5: /Motortreiber5/MA1 -> /Motortreiber8/MA1
- U1501 pad 6: Net-(U1501-Pad6) -> (no net)
- U1601 pad 1: +28V -> Net-(C1601-Pad1)
- U1601 pad 16: Net-(C1602-Pad1) -> Net-(C1603-Pad1)
- U1601 pad 17: /Steuer5 -> Net-(C1604-Pad1)
- U1601 pad 18: /Steuer6 -> Net-(C1606-Pad1)
- U1601 pad 19: Net-(U1601-Pad19) -> (no net)
- U1601 pad 2: +28V -> Net-(C1601-Pad1)
- U1601 pad 20: /Motortreiber6/MD2 -> /Motortreiber4/MD2
- U1601 pad 21: /Motortreiber6/MDR -> /Motortreiber4/MDR
- U1601 pad 22: /Motortreiber6/MD1 -> /Motortreiber4/MD1
- U1601 pad 23: +28V -> Net-(C1601-Pad1)
- U1601 pad 24: +28V -> Net-(C1601-Pad1)
- U1601 pad 25: /Motortreiber6/MC2 -> /Motortreiber4/MC2
- U1601 pad 26: /Motortreiber6/MCR -> /Motortreiber4/MCR
- U1601 pad 27: /Motortreiber6/MC1 -> /Motortreiber4/MC1
- U1601 pad 28: Net-(U1601-Pad28) -> (no net)
- U1601 pad 29: Net-(U1601-Pad29) -> (no net)
- U1601 pad 3: /Motortreiber6/MA2 -> /Motortreiber4/MA2
- U1601 pad 30: /Strobe6 -> /Strobe4
- U1601 pad 32: Net-(U1601-Pad32) -> (no net)
- U1601 pad 4: /Motortreiber6/MAR -> /Motortreiber4/MAR
- U1601 pad 40: Net-(U1601-Pad40) -> (no net)
- U1601 pad 41: Net-(U1601-Pad41) -> (no net)
- U1601 pad 44: Net-(U1601-Pad44) -> (no net)
- U1601 pad 46: /Motortreiber6/MB1 -> /Motortreiber4/MB1
- U1601 pad 47: /Motortreiber6/MBR -> /Motortreiber4/MBR
- U1601 pad 48: /Motortreiber6/MB2 -> /Motortreiber4/MB2
- U1601 pad 5: /Motortreiber6/MA1 -> /Motortreiber4/MA1
- U1601 pad 6: Net-(U1601-Pad6) -> (no net)
- U1701 pad 1: +28V -> Net-(C1701-Pad1)
- U1701 pad 16: Net-(C1702-Pad1) -> Net-(C1703-Pad1)
- U1701 pad 17: /Steuer5 -> Net-(C1704-Pad1)
- U1701 pad 18: /Steuer6 -> Net-(C1706-Pad1)
- U1701 pad 19: Net-(U1701-Pad19) -> (no net)
- U1701 pad 2: +28V -> Net-(C1701-Pad1)
- U1701 pad 20: /Motortreiber7/MD2 -> /Motortreiber10/MD2
- U1701 pad 21: /Motortreiber7/MDR -> /Motortreiber10/MDR
- U1701 pad 22: /Motortreiber7/MD1 -> /Motortreiber10/MD1
- U1701 pad 23: +28V -> Net-(C1701-Pad1)
- U1701 pad 24: +28V -> Net-(C1701-Pad1)
- U1701 pad 25: /Motortreiber7/MC2 -> /Motortreiber10/MC2
- U1701 pad 26: /Motortreiber7/MCR -> /Motortreiber10/MCR
- U1701 pad 27: /Motortreiber7/MC1 -> /Motortreiber10/MC1
- U1701 pad 28: Net-(U1701-Pad28) -> (no net)
- U1701 pad 29: Net-(U1701-Pad29) -> (no net)
- U1701 pad 3: /Motortreiber7/MA2 -> /Motortreiber10/MA2
- U1701 pad 30: /Strobe7 -> /Strobe10
- U1701 pad 32: Net-(U1701-Pad32) -> (no net)
- U1701 pad 4: /Motortreiber7/MAR -> /Motortreiber10/MAR
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Routing:
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- added copper zone on B.Cu, net GND
- added copper zone on F.Cu, net GND
Other:
- board size 200 x 300 mm -> 200.7 x 279.4 mm
- board text added: "5"
